File: sequencer.sch (KiCad schematic (older format))
At the start: 14 parts, among them J101 USB_A, J102 NHD-3.12-25664UC, J103 PJS008U-3000, U101 74HCT541, U102 74HC595, U103 74HC595, U104 74HC595, U105 74HC165

Commit message: work on schematic
Connections:
- net GND: now also J101.4 (GND), J101.5 (Shield)
- net USB_5V: now reaches J101.1 (VBUS)
- net USB_DM: now reaches J101.2 (D-)
- net USB_DP: now reaches J101.3 (D+)
Other:
- moved on the sheet: J101
Changed lines of the file:
@@
 EESchema Schematic File Version 2
+LIBS:w_power
 LIBS:w_lcd
 LIBS:w_stm32
@@
 encoding utf-8
 Sheet 1 7
-Title ""
+Title "Eurorack Sequencer"
 Date ""
-Rev ""
-Comp ""
+Rev "0.1"
+Comp "westlicht"
 Comment1 ""
 Comment2 ""
@@
 L USB_A J101
 U 1 1 59DE5EB2
-P 3450 3700
-F 0 "J101" H 3250 4150 50  0000 L CNN
-F 1 "USB_A" H 3250 4050 50  0000 L CNN
-F 2 "w_connector:MOLEX_USB_105057" H 3600 3650 50  0001 C CNN
-F 3 "http://datasheet.octopart.com/105057-0001-Molex-datasheet-48881000.pdf" H 3600 3650 50  0001 C CNN
-F 4 "test" H 3450 3700 60  0001 C CNN "Description"
-F 5 "Molex" H 3450 3700 60  0001 C CNN "MFN"
-F 6 "105057-0001" H 3450 3700 60  0001 C CNN "MFP"
-	1    3450 3700
+P 3500 3700
+F 0 "J101" H 3300 4150 50  0000 L CNN
+F 1 "USB_A" H 3300 4050 50  0000 L CNN
+F 2 "w_connector:MOLEX_USB_105057" H 3650 3650 50  0001 C CNN
+F 3 "http://datasheet.octopart.com/105057-0001-Molex-datasheet-48881000.pdf" H 3650 3650 50  0001 C CNN
+F 4 "test" H 3500 3700 60  0001 C CNN "Description"
+F 5 "Molex" H 3500 3700 60  0001 C CNN "MFN"
+F 6 "105057-0001" H 3500 3700 60  0001 C CNN "MFP"
+	1    3500 3700
 	1    0    0    -1
 $EndComp
@@
 NoConn ~ 9200 2000
 NoConn ~ 9200 1300
+Text GLabel 3900 3500 2    51   Input ~ 0
+USB_5V
+Wire Wire Line
+	3900 3500 3800 3500
+Text GLabel 3900 3700 2    51   Input ~ 0
+USB_DP
+Text GLabel 3900 3800 2    51   Input ~ 0
+USB_DM
+Wire Wire Line
+	3800 3700 3900 3700
+Wire Wire Line
+	3800 3800 3900 3800
+Wire Wire Line
+	3500 4100 3500 4300
+$Comp
+L GND #PWR021
+U 1 1 59E06450
+P 3500 4300
+F 0 "#PWR021" H 3500 4050 50  0001 C CNN
+F 1 "GND" H 3500 4150 50  0000 C CNN
+F 2 "" H 3500 4300 50  0001 C CNN
+F 3 "" H 3500 4300 50  0001 C CNN
+	1    3500 4300
+	1    0    0    -1
+$EndComp
+Wire Wire Line
+	3400 4100 3400 4200
+Wire Wire Line
+	3400 4200 3500 4200
+Connection ~ 3500 4200
 $EndSCHEMATC

Commit message: work in progress
Parts:
- C101, C102, C103, C104, C105: MFN (none) -> Murata; MFP (none) -> GRM188R71E104JA01J
- J101: Description test -> (none)
- U102, U103, U104, U105: footprint Housings_SSOP:TSSOP-16_4.4x5mm_Pitch0.65mm -> Housings_SOIC:SOIC-16_3.9x9.9mm_Pitch1.27mm
Changed lines of the file:
@@
 F 1 "ALPS-STEC12E08" H 3050 7000 50  0000 C CNN
 F 2 "w_rotary_encoder:ALPS_STEC12E08" H 3050 6650 60  0001 C CNN
-F 3 "" H 3050 6650 60  0000 C CNN
+F 3 "http://datasheet.octopart.com/PEC11R-4225F-S0024-Bourns-datasheet-68303416.pdf" H 3050 6650 60  0001 C CNN
 F 4 "Bourns" H 3050 6400 50  0001 C CNN "MFN"
 F 5 "PEC11R-4225F-S0024" H 3050 6400 50  0001 C CNN "MFP"
@@
 F 0 "U105" H 7100 4250 60  0000 C CNN
 F 1 "74HC165" H 7100 5250 60  0000 C CNN
-F 2 "Housings_SSOP:TSSOP-16_4.4x5mm_Pitch0.65mm" H 6600 5100 60  0001 C CNN
+F 2 "Housings_SOIC:SOIC-16_3.9x9.9mm_Pitch1.27mm" H 6600 5100 60  0001 C CNN
 F 3 "" H 6600 5100 60  0001 C CNN
 	1    6600 5100
@@
 F 0 "U102" H 7100 50  60  0000 C CNN
 F 1 "74HC595" H 7100 1050 60  0000 C CNN
-F 2 "Housings_SSOP:TSSOP-16_4.4x5mm_Pitch0.65mm" H 6600 900 60  0001 C CNN
+F 2 "Housings_SOIC:SOIC-16_3.9x9.9mm_Pitch1.27mm" H 6600 900 60  0001 C CNN
 F 3 "" H 6600 900 60  0001 C CNN
 	1    6600 900
@@
 F 0 "U103" H 7100 1450 60  0000 C CNN
 F 1 "74HC595" H 7100 2450 60  0000 C CNN
-F 2 "Housings_SSOP:TSSOP-16_4.4x5mm_Pitch0.65mm" H 6600 2300 60  0001 C CNN
+F 2 "Housings_SOIC:SOIC-16_3.9x9.9mm_Pitch1.27mm" H 6600 2300 60  0001 C CNN
 F 3 "" H 6600 2300 60  0001 C CNN
 	1    6600 2300
@@
 F 0 "U104" H 7100 2850 60  0000 C CNN
 F 1 "74HC595" H 7100 3850 60  0000 C CNN
-F 2 "Housings_SSOP:TSSOP-16_4.4x5mm_Pitch0.65mm" H 6600 3700 60  0001 C CNN
+F 2 "Housings_SOIC:SOIC-16_3.9x9.9mm_Pitch1.27mm" H 6600 3700 60  0001 C CNN
 F 3 "" H 6600 3700 60  0001 C CNN
 	1    6600 3700
@@
 F 1 "100n" H 5025 6750 50  0000 L CNN
 F 2 "Capacitors_SMD:C_0603" H 5038 6700 50  0001 C CNN
-F 3 "" H 5000 6850 50  0001 C CNN
+F 3 "http://datasheet.octopart.com/GRM188R71E104JA01J-Murata-datasheet-66077098.pdf" H 5000 6850 50  0001 C CNN
+F 4 "Murata" H 5025 7050 50  0001 C CNN "MFN"
+F 5 "GRM188R71E104JA01J" H 5025 7050 50  0001 C CNN "MFP"
 	1    5000 6850
 	1    0    0    -1
@@
 F 1 "100n" H 5325 6750 50  0000 L CNN
 F 2 "Capacitors_SMD:C_0603" H 5338 6700 50  0001 C CNN
-F 3 "" H 5300 6850 50  0001 C CNN
+F 3 "http://datasheet.octopart.com/GRM188R71E104JA01J-Murata-datasheet-66077098.pdf" H 5300 6850 50  0001 C CNN
+F 4 "Murata" H 5325 7050 50  0001 C CNN "MFN"
+F 5 "GRM188R71E104JA01J" H 5325 7050 50  0001 C CNN "MFP"
 	1    5300 6850
 	1    0    0    -1
@@
 F 1 "100n" H 5625 6750 50  0000 L CNN
 F 2 "Capacitors_SMD:C_0603" H 5638 6700 50  0001 C CNN
-F 3 "" H 5600 6850 50  0001 C CNN
+F 3 "http://datasheet.octopart.com/GRM188R71E104JA01J-Murata-datasheet-66077098.pdf" H 5600 6850 50  0001 C CNN
+F 4 "Murata" H 5625 7050 50  0001 C CNN "MFN"
+F 5 "GRM188R71E104JA01J" H 5625 7050 50  0001 C CNN "MFP"
 	1    5600 6850
 	1    0    0    -1
@@
 F 1 "100n" H 5925 6750 50  0000 L CNN
 F 2 "Capacitors_SMD:C_0603" H 5938 6700 50  0001 C CNN
-F 3 "" H 5900 6850 50  0001 C CNN
+F 3 "http://datasheet.octopart.com/GRM188R71E104JA01J-Murata-datasheet-66077098.pdf" H 5900 6850 50  0001 C CNN
+F 4 "Murata" H 5925 7050 50  0001 C CNN "MFN"
+F 5 "GRM188R71E104JA01J" H 5925 7050 50  0001 C CNN "MFP"
 	1    5900 6850
 	1    0    0    -1
@@
 F 1 "100n" H 6225 6750 50  0000 L CNN
 F 2 "Capacitors_SMD:C_0603" H 6238 6700 50  0001 C CNN
-F 3 "" H 6200 6850 50  0001 C CNN
+F 3 "http://datasheet.octopart.com/GRM188R71E104JA01J-Murata-datasheet-66077098.pdf" H 6200 6850 50  0001 C CNN
+F 4 "Murata" H 6225 7050 50  0001 C CNN "MFN"
+F 5 "GRM188R71E104JA01J" H 6225 7050 50  0001 C CNN "MFP"
 	1    6200 6850
 	1    0    0    -1
@@
 F 2 "w_connector:MOLEX_USB_105057" H 3650 3650 50  0001 C CNN
 F 3 "http://datasheet.octopart.com/105057-0001-Molex-datasheet-48881000.pdf" H 3650 3650 50  0001 C CNN
-F 4 "test" H 3500 3700 60  0001 C CNN "Description"
-F 5 "Molex" H 3500 3700 60  0001 C CNN "MFN"
-F 6 "105057-0001" H 3500 3700 60  0001 C CNN "MFP"
+F 4 "Molex" H 3500 3700 60  0001 C CNN "MFN"
+F 5 "105057-0001" H 3500 3700 60  0001 C CNN "MFP"
 	1    3500 3700
+	1    0    0    -1
+$EndComp
+$Comp
+L GND #PWR021
+U 1 1 59E06450
+P 3500 4300
+F 0 "#PWR021" H 3500 4050 50  0001 C CNN
+F 1 "GND" H 3500 4150 50  0000 C CNN
+F 2 "" H 3500 4300 50  0001 C CNN
+F 3 "" H 3500 4300 50  0001 C CNN
+	1    3500 4300
 	1    0    0    -1
 $EndComp
@@
 Text GLabel 2400 6500 0    51   Output ~ 0
 ENC_SW
+Text GLabel 3900 3500 2    51   Input ~ 0
+USB_5V
+Text GLabel 3900 3700 2    51   Input ~ 0
+USB_DP
+Text GLabel 3900 3800 2    51   Input ~ 0
+USB_DM
 Wire Wire Line
 	7600 900  7700 900
@@
 Wire Wire Line
 	2400 6800 2400 7050
+Wire Wire Line
+	3900 3500 3800 3500
+Wire Wire Line
+	3800 3700 3900 3700
+Wire Wire Line
+	3800 3800 3900 3800
+Wire Wire Line
+	3500 4100 3500 4300
+Wire Wire Line
+	3400 4100 3400 4200
+Wire Wire Line
+	3400 4200 3500 4200
 Connection ~ 6500 1600
 Connection ~ 6500 3000
@@
 Connection ~ 9400 4900
 Connection ~ 9400 5000
+Connection ~ 3500 4200
 NoConn ~ 6600 5400
 NoConn ~ 5100 1500
@@
 NoConn ~ 9200 2000
 NoConn ~ 9200 1300
-Text GLabel 3900 3500 2    51   Input ~ 0
-USB_5V
-Wire Wire Line
-	3900 3500 3800 3500
-Text GLabel 3900 3700 2    51   Input ~ 0
-USB_DP
-Text GLabel 3900 3800 2    51   Input ~ 0
-USB_DM
-Wire Wire Line
-	3800 3700 3900 3700
-Wire Wire Line
-	3800 3800 3900 3800
-Wire Wire Line
-	3500 4100 3500 4300
-$Comp
-L GND #PWR021
-U 1 1 59E06450
-P 3500 4300
-F 0 "#PWR021" H 3500 4050 50  0001 C CNN
-F 1 "GND" H 3500 4150 50  0000 C CNN
-F 2 "" H 3500 4300 50  0001 C CNN
-F 3 "" H 3500 4300 50  0001 C CNN
-	1    3500 4300
-	1    0    0    -1
-$EndComp
-Wire Wire Line
-	3400 4100 3400 4200
-Wire Wire Line
-	3400 4200 3500 4200
-Connection ~ 3500 4200
 $EndSCHEMATC

Commit message: more work
Parts:
- U102, U103, U104: MFN (none) -> Texas Instruments; MFP (none) -> SN74HC595D
- U105: MFN (none) -> Texas Instruments; MFP (none) -> SN74HC165D
Changed lines of the file:
@@
 F 1 "74HC165" H 7100 5250 60  0000 C CNN
 F 2 "Housings_SOIC:SOIC-16_3.9x9.9mm_Pitch1.27mm" H 6600 5100 60  0001 C CNN
-F 3 "" H 6600 5100 60  0001 C CNN
+F 3 "https://octopart.com/click/track?ct=datasheets&hlid=24916538&ppid=35776&sid=370&sig=03765d0" H 6600 5100 60  0001 C CNN
+F 4 "Texas Instruments" H 7100 4350 50  0001 C CNN "MFN"
+F 5 "SN74HC165D" H 7100 4350 50  0001 C CNN "MFP"
 	1    6600 5100
 	1    0    0    -1
@@
 F 1 "74HC595" H 7100 1050 60  0000 C CNN
 F 2 "Housings_SOIC:SOIC-16_3.9x9.9mm_Pitch1.27mm" H 6600 900 60  0001 C CNN
-F 3 "" H 6600 900 60  0001 C CNN
+F 3 "https://octopart.com/click/track?ct=datasheets&hlid=24917219&ppid=44183&sid=370&sig=036bbbe" H 6600 900 60  0001 C CNN
+F 4 "Texas Instruments" H 7100 150 50  0001 C CNN "MFN"
+F 5 "SN74HC595D" H 7100 150 50  0001 C CNN "MFP"
 	1    6600 900
 	1    0    0    -1
@@
 F 1 "74HC595" H 7100 2450 60  0000 C CNN
 F 2 "Housings_SOIC:SOIC-16_3.9x9.9mm_Pitch1.27mm" H 6600 2300 60  0001 C CNN
-F 3 "" H 6600 2300 60  0001 C CNN
+F 3 "https://octopart.com/click/track?ct=datasheets&hlid=24917219&ppid=44183&sid=370&sig=036bbbe" H 6600 2300 60  0001 C CNN
+F 4 "Texas Instruments" H 7100 1550 50  0001 C CNN "MFN"
+F 5 "SN74HC595D" H 7100 1550 50  0001 C CNN "MFP"
 	1    6600 2300
 	1    0    0    -1
@@
 F 1 "74HC595" H 7100 3850 60  0000 C CNN
 F 2 "Housings_SOIC:SOIC-16_3.9x9.9mm_Pitch1.27mm" H 6600 3700 60  0001 C CNN
-F 3 "" H 6600 3700 60  0001 C CNN
+F 3 "https://octopart.com/click/track?ct=datasheets&hlid=24917219&ppid=44183&sid=370&sig=036bbbe" H 6600 3700 60  0001 C CNN
+F 4 "Texas Instruments" H 7100 2950 50  0001 C CNN "MFN"
+F 5 "SN74HC595D" H 7100 2950 50  0001 C CNN "MFP"
 	1    6600 3700
 	1    0    0    -1

Commit message: work in progress
Parts:
- removed U101: 74HCT541, Housings_SOIC:SOIC-20W_7.5x12.8mm_Pitch1.27mm, symbol 74HCT541
- added R101, R102, R103, R104, R105: 10k, Resistors_SMD:R_0603, symbol R
- added R106, R107, R108, R109, R110, R111, R112, R113: 470, Resistors_SMD:R_0603, symbol R
- added U101: 74HCT125, Housings_SOIC:SOIC-14_3.9x8.7mm_Pitch1.27mm, symbol 74HCT125
Connections:
- net +5V: now also R101.1, R102.1, R103.1, R104.1, R105.1, U101.14 (VCC)
- net ENC_SW: no longer ENC101.SW1
- net GCOL0: now also R107.1; no longer U103.1 (QB)
- net GCOL1: now also R109.1; no longer U103.3 (QD)
- net GCOL2: now also R111.1; no longer U103.5 (QF)
- net GCOL3: now also R113.1; no longer U103.7 (QH)
- net GND: now also U101.1 (1~OE), U101.10 (3~OE), U101.13 (4~OE), U101.4 (2~OE), U101.7 (GND); no longer ENC101.SW2
- net RCOL0: now also R106.1; no longer U103.10 (QA)
- net RCOL1: now also R108.1; no longer U103.2 (QC)
- net RCOL2: now also R110.1; no longer U103.4 (QE)
- net RCOL3: now also R112.1; no longer U103.6 (QG)
- net SCOL0: now also R101.2
- net SCOL1: now also R102.2
- net SCOL2: now also R103.2
- net SCOL3: now also R104.2
- net SCOL4: now also R105.2
- net SR_LATCH: now also U101.9 (3A)
- net SR_LOAD: now also U101.12 (4A)
- net SR_MOSI: now also U101.2 (1A)
- net SR_SCK: now also U101.5 (2A)
- net at U105.1 (~LD~): now also U101.11 (4Y)
- net at U102.14 (SRCLK), U103.14 (SRCLK), U104.14 (SRCLK)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: now also U101.6 (2Y)
- net at U102.11 (SER): now also U101.3 (1Y)
- net at U102.13 (RCLK), U103.13 (RCLK), U104.13 (RCLK): now also U101.8 (3Y)
- new net: R107.2, U103.1 (QB)
- new net: R106.2, U103.10 (QA)
- new net: R108.2, U103.2 (QC)
- new net: R109.2, U103.3 (QD)
- new net: R110.2, U103.4 (QE)
- new net: R111.2, U103.5 (QF)
- new net: R112.2, U103.6 (QG)
- new net: R113.2, U103.7 (QH)
- no-connect marks 7 -> 3
Other:
- moved on the sheet: J101, J102, J103, U102, U103, U104, U105

Commit message: more work on layout
Connections:
- net ENC_SW: now also ENC101.SW1
- net GND: now also ENC101.SW2
- net USB_DM renamed USB_D-
- net USB_DP renamed USB_D+
Changed lines of the file:
@@
 L GND #PWR018
 U 1 1 59DDDDF7
-P 3500 7050
-F 0 "#PWR018" H 3500 6800 50  0001 C CNN
-F 1 "GND" H 3500 6900 50  0000 C CNN
-F 2 "" H 3500 7050 50  0001 C CNN
-F 3 "" H 3500 7050 50  0001 C CNN
-	1    3500 7050
+P 2400 7050
+F 0 "#PWR018" H 2400 6800 50  0001 C CNN
+F 1 "GND" H 2400 6900 50  0000 C CNN
+F 2 "" H 2400 7050 50  0001 C CNN
+F 3 "" H 2400 7050 50  0001 C CNN
+	1    2400 7050
 	1    0    0    -1
 $EndComp
@@
 Text GLabel 3800 6900 2    51   Output ~ 0
 ENC_B
-Text GLabel 3500 6500 0    51   Output ~ 0
+Text GLabel 2400 6500 0    51   Output ~ 0
 ENC_SW
 Text GLabel 10400 5400 2    51   Input ~ 0
 USB_5V
 Text GLabel 10400 5600 2    51   Input ~ 0
-USB_DP
+USB_D+
 Text GLabel 10400 5700 2    51   Input ~ 0
-USB_DM
+USB_D-
 Wire Wire Line
 	6500 900  6600 900
@@
 	3600 6400 3800 6400
 Wire Wire Line
-	3500 6500 3600 6500
-Wire Wire Line
-	3600 6800 3500 6800
-Wire Wire Line
-	3500 6800 3500 7050
+	2400 6500 2500 6500
+Wire Wire Line
+	2500 6800 2400 6800
+Wire Wire Line
+	2400 6800 2400 7050
 Wire Wire Line
 	10400 5400 10300 5400

Commit message: redesign in progress
Parts:
- R101, R102, R103, R104, R105: MFN (none) -> Panasonic; MFP (none) -> ERJ-3EKF1002V
- R106, R107, R108, R109, R110, R111, R112, R113: MFN (none) -> Panasonic; MFP (none) -> ERJ-3EKF4700V
- U101: MFN Texas Instruments -> Texas Instruments

Commit message: only ground plane left
Connections:
- net GND: no longer U105.9 (QH)
- no-connect marks 3 -> 5
Changed lines of the file:
@@
 $EndComp
 $Comp
-L GND #PWR112
+L GND #PWR01
 U 1 1 59DAC8B2
 P 5400 4500
-F 0 "#PWR112" H 5400 4250 50  0001 C CNN
+F 0 "#PWR01" H 5400 4250 50  0001 C CNN
 F 1 "GND" H 5400 4350 50  0000 C CNN
 F 2 "" H 5400 4500 50  0001 C CNN
@@
 $EndComp
 $Comp
-L GND #PWR110
+L GND #PWR02
 U 1 1 59DAC8DB
 P 5400 3100
-F 0 "#PWR110" H 5400 2850 50  0001 C CNN
+F 0 "#PWR02" H 5400 2850 50  0001 C CNN
 F 1 "GND" H 5400 2950 50  0000 C CNN
 F 2 "" H 5400 3100 50  0001 C CNN
@@
 $EndComp
 $Comp
-L GND #PWR104
+L GND #PWR03
 U 1 1 59DAC904
 P 5400 1700
-F 0 "#PWR104" H 5400 1450 50  0001 C CNN
+F 0 "#PWR03" H 5400 1450 50  0001 C CNN
 F 1 "GND" H 5400 1550 50  0000 C CNN
 F 2 "" H 5400 1700 50  0001 C CNN
@@
 $EndComp
 $Comp
-L +5V #PWR102
+L +5V #PWR04
 U 1 1 59DACCD2
 P 5300 800
-F 0 "#PWR102" H 5300 650 50  0001 C CNN
+F 0 "#PWR04" H 5300 650 50  0001 C CNN
 F 1 "+5V" H 5300 940 50  0000 C CNN
 F 2 "" H 5300 800 50  0001 C CNN
@@
 $EndComp
 $Comp
-L +5V #PWR108
+L +5V #PWR05
 U 1 1 59DACCFB
 P 5300 2200
-F 0 "#PWR108" H 5300 2050 50  0001 C CNN
+F 0 "#PWR05" H 5300 2050 50  0001 C CNN
 F 1 "+5V" H 5300 2340 50  0000 C CNN
 F 2 "" H 5300 2200 50  0001 C CNN
@@
 $EndComp
 $Comp
-L +5V #PWR111
+L +5V #PWR06
 U 1 1 59DACD24
 P 5300 3600
-F 0 "#PWR111" H 5300 3450 50  0001 C CNN
+F 0 "#PWR06" H 5300 3450 50  0001 C CNN
 F 1 "+5V" H 5300 3740 50  0000 C CNN
 F 2 "" H 5300 3600 50  0001 C CNN
@@
 $EndComp
 $Comp
-L GND #PWR116
+L GND #PWR07
 U 1 1 59DADBC6
 P 5400 5900
-F 0 "#PWR116" H 5400 5650 50  0001 C CNN
+F 0 "#PWR07" H 5400 5650 50  0001 C CNN
 F 1 "GND" H 5400 5750 50  0000 C CNN
 F 2 "" H 5400 5900 50  0001 C CNN
@@
 $EndComp
 $Comp
-L +5V #PWR115
+L +5V #PWR08
 U 1 1 59DADC53
 P 5300 5000
-F 0 "#PWR115" H 5300 4850 50  0001 C CNN
+F 0 "#PWR08" H 5300 4850 50  0001 C CNN
 F 1 "+5V" H 5300 5140 50  0000 C CNN
 F 2 "" H 5300 5000 50  0001 C CNN
@@
 $EndComp
 $Comp
-L GND #PWR117
+L GND #PWR09
 U 1 1 59DAEC89
 P 6600 5900
-F 0 "#PWR117" H 6600 5650 50  0001 C CNN
+F 0 "#PWR09" H 6600 5650 50  0001 C CNN
 F 1 "GND" H 6600 5750 50  0000 C CNN
 F 2 "" H 6600 5900 50  0001 C CNN
@@
 $EndComp
 $Comp
-L +5V #PWR119
+L +5V #PWR010
 U 1 1 59DB575D
 P 4900 6500
-F 0 "#PWR119" H 4900 6350 50  0001 C CNN
+F 0 "#PWR010" H 4900 6350 50  0001 C CNN
 F 1 "+5V" H 4900 6640 50  0000 C CNN
 F 2 "" H 4900 6500 50  0001 C CNN
@@
 $EndComp
 $Comp
-L GND #PWR122
+L GND #PWR011
 U 1 1 59DB5795
 P 4900 7200
-F 0 "#PWR122" H 4900 6950 50  0001 C CNN
+F 0 "#PWR011" H 4900 6950 50  0001 C CNN
 F 1 "GND" H 4900 7050 50  0000 C CNN
 F 2 "" H 4900 7200 50  0001 C CNN
@@
 $EndComp
 $Comp
-L +3.3V #PWR103
+L +3.3V #PWR012
 U 1 1 59DD8249
 P 9000 900
-F 0 "#PWR103" H 9000 750 50  0001 C CNN
+F 0 "#PWR012" H 9000 750 50  0001 C CNN
 F 1 "+3.3V" H 9000 1040 50  0000 C CNN
 F 2 "" H 9000 900 50  0001 C CNN
@@
 $EndComp
 $Comp
-L GND #PWR106
+L GND #PWR013
 U 1 1 59DD828A
 P 9100 2000
-F 0 "#PWR106" H 9100 1750 50  0001 C CNN
+F 0 "#PWR013" H 9100 1750 50  0001 C CNN
 F 1 "GND" H 9100 1850 50  0000 C CNN
 F 2 "" H 9100 2000 50  0001 C CNN
@@
 $EndComp
 $Comp
-L GND #PWR107
+L GND #PWR014
 U 1 1 59DD85C7
 P 11000 2100
-F 0 "#PWR107" H 11000 1850 50  0001 C CNN
+F 0 "#PWR014" H 11000 1850 50  0001 C CNN
 F 1 "GND" H 11000 1950 50  0000 C CNN
 F 2 "" H 11000 2100 50  0001 C CNN
@@
 $EndComp
 $Comp
-L GND #PWR114
+L GND #PWR015
 U 1 1 59DDC96B
 P 9400 4800
-F 0 "#PWR114" H 9400 4550 50  0001 C CNN
+F 0 "#PWR015" H 9400 4550 50  0001 C CNN
 F 1 "GND" H 9400 4650 50  0000 C CNN
 F 2 "" H 9400 4800 50  0001 C CNN
@@
 $EndComp
 $Comp
-L +3.3V #PWR109
+L +3.3V #PWR016
 U 1 1 59DDCA82
 P 9300 2700
-F 0 "#PWR109" H 9300 2550 50  0001 C CNN
+F 0 "#PWR016" H 9300 2550 50  0001 C CNN
 F 1 "+3.3V" H 9300 2840 50  0000 C CNN
 F 2 "" H 9300 2700 50  0001 C CNN
@@
 $EndComp
 $Comp
-L GND #PWR121
+L GND #PWR017
 U 1 1 59DDD81F
 P 3700 7050
-F 0 "#PWR121" H 3700 6800 50  0001 C CNN
+F 0 "#PWR017" H 3700 6800 50  0001 C CNN
 F 1 "GND" H 3700 6900 50  0000 C CNN
 F 2 "" H 3700 7050 50  0001 C CNN
@@
 $EndComp
 $Comp
-L GND #PWR120
+L GND #PWR018
 U 1 1 59DDDDF7
 P 2400 7050
-F 0 "#PWR120" H 2400 6800 50  0001 C CNN
+F 0 "#PWR018" H 2400 6800 50  0001 C CNN
 F 1 "GND" H 2400 6900 50  0000 C CNN
 F 2 "" H 2400 7050 50  0001 C CNN
@@
 $EndComp
 $Comp
-L GND #PWR118
+L GND #PWR019
 U 1 1 59E06450
 P 10000 6200
-F 0 "#PWR118" H 10000 5950 50  0001 C CNN
+F 0 "#PWR019" H 10000 5950 50  0001 C CNN
 F 1 "GND" H 10000 6050 50  0000 C CNN
 F 2 "" H 10000 6200 50  0001 C CNN
@@
 $EndComp
 $Comp
-L +5V #PWR113
+L +5V #PWR020
 U 1 1 59E571E6
 P 7600 4500
-F 0 "#PWR113" H 7600 4350 50  0001 C CNN
+F 0 "#PWR020" H 7600 4350 50  0001 C CNN
 F 1 "+5V" H 7600 4640 50  0000 C CNN
 F 2 "" H 7600 4500 50  0001 C CNN
@@
 $EndComp
 $Comp
-L GND #PWR105
+L GND #PWR021
 U 1 1 59E5F67D
 P 2900 1800
-F 0 "#PWR105" H 2900 1550 50  0001 C CNN
+F 0 "#PWR021" H 2900 1550 50  0001 C CNN
 F 1 "GND" H 2900 1650 50  0000 C CNN
 F 2 "" H 2900 1800 50  0001 C CNN
@@
 $EndComp
 $Comp
-L +5V #PWR101
+L +5V #PWR022
 U 1 1 59E5F6E5
 P 2900 700
-F 0 "#PWR101" H 2900 550 50  0001 C CNN
+F 0 "#PWR022" H 2900 550 50  0001 C CNN
 F 1 "+5V" H 2900 840 50  0000 C CNN
 F 2 "" H 2900 700 50  0001 C CNN
@@
 	5400 5800 5500 5800
 Wire Wire Line
-	5400 5500 5400 5900
-Wire Wire Line
 	5300 5000 5300 5100
 Wire Wire Line
@@
 Wire Wire Line
 	5500 5700 5400 5700
-Wire Wire Line
-	5500 5500 5400 5500
 Wire Wire Line
 	5100 5300 5500 5300
@@
 Connection ~ 6600 5700
 Connection ~ 6600 5800
-Connection ~ 5400 5800
-Connection ~ 5400 5700
 Connection ~ 5900 7100
 Connection ~ 5900 6600
@@
 NoConn ~ 9200 1800
 NoConn ~ 9200 1100
+Wire Wire Line
+	5400 5700 5400 5900
+Connection ~ 5400 5800
+NoConn ~ 5500 5500
+NoConn ~ 5500 4300
 $EndSCHEMATC
