File: mcu.sch (KiCad schematic (older format))
At the start: 12 parts, among them J501 JTAG, J502 Serial / Bootloader, SW501 EVQQ2, SW502 EVQQ2, U501 STM32F405RGTx, Y501 8MHz

Commit message: work on schematic
Connections:
- net USB_DM: now reaches U501.44 (ADC1_EXTI11/ADC2_EXTI11/ADC3_EXTI11/CAN1_RX/TIM1_CH4/USART1_CTS/USB_OTG_FS_DM/PA11)
- net USB_DP: now reaches U501.45 (CAN1_TX/TIM1_ETR/USART1_RTS/USB_OTG_FS_DP/PA12)
Changed lines of the file:
@@
 EESchema Schematic File Version 2
+LIBS:w_power
 LIBS:w_lcd
 LIBS:w_stm32
@@
 encoding utf-8
 Sheet 5 7
-Title ""
+Title "Eurorack Sequencer"
 Date ""
-Rev ""
-Comp ""
+Rev "0.1"
+Comp "westlicht"
 Comment1 ""
 Comment2 ""
@@
 $EndComp
 $Comp
-L GND #PWR039
+L GND #PWR049
 U 1 1 59DB9615
 P 1600 6500
-F 0 "#PWR039" H 1600 6250 50  0001 C CNN
+F 0 "#PWR049" H 1600 6250 50  0001 C CNN
 F 1 "GND" H 1600 6350 50  0000 C CNN
 F 2 "" H 1600 6500 50  0001 C CNN
@@
 $EndComp
 $Comp
-L +3.3V #PWR040
+L +3.3V #PWR050
 U 1 1 59DB9CCC
 P 2500 5800
-F 0 "#PWR040" H 2500 5650 50  0001 C CNN
+F 0 "#PWR050" H 2500 5650 50  0001 C CNN
 F 1 "+3.3V" H 2500 5940 50  0000 C CNN
 F 2 "" H 2500 5800 50  0001 C CNN
@@
 $EndComp
 $Comp
-L GND #PWR041
+L GND #PWR051
 U 1 1 59DB9CF4
 P 2500 6400
-F 0 "#PWR041" H 2500 6150 50  0001 C CNN
+F 0 "#PWR051" H 2500 6150 50  0001 C CNN
 F 1 "GND" H 2500 6250 50  0000 C CNN
 F 2 "" H 2500 6400 50  0001 C CNN
@@
 $EndComp
 $Comp
-L +3.3V #PWR042
+L +3.3V #PWR052
 U 1 1 59DB9EAC
 P 5500 1000
-F 0 "#PWR042" H 5500 850 50  0001 C CNN
+F 0 "#PWR052" H 5500 850 50  0001 C CNN
 F 1 "+3.3V" H 5500 1140 50  0000 C CNN
 F 2 "" H 5500 1000 50  0001 C CNN
@@
 $EndComp
 $Comp
-L +3.3VA #PWR043
+L +3.3VA #PWR053
 U 1 1 59DB9EE7
 P 6000 1000
-F 0 "#PWR043" H 6000 850 50  0001 C CNN
+F 0 "#PWR053" H 6000 850 50  0001 C CNN
 F 1 "+3.3VA" H 6000 1140 50  0000 C CNN
 F 2 "" H 6000 1000 50  0001 C CNN
@@
 $EndComp
 $Comp
-L GND #PWR044
+L GND #PWR054
 U 1 1 59DB9FE7
 P 5800 5400
-F 0 "#PWR044" H 5800 5150 50  0001 C CNN
+F 0 "#PWR054" H 5800 5150 50  0001 C CNN
 F 1 "GND" H 5800 5250 50  0000 C CNN
 F 2 "" H 5800 5400 50  0001 C CNN
@@
 $EndComp
 $Comp
-L GND #PWR045
+L GND #PWR055
 U 1 1 59DBA437
 P 800 7500
-F 0 "#PWR045" H 800 7250 50  0001 C CNN
+F 0 "#PWR055" H 800 7250 50  0001 C CNN
 F 1 "GND" H 800 7350 50  0000 C CNN
 F 2 "" H 800 7500 50  0001 C CNN
@@
 $EndComp
 $Comp
-L GND #PWR046
+L GND #PWR056
 U 1 1 59DBB736
 P 800 2250
-F 0 "#PWR046" H 800 2000 50  0001 C CNN
+F 0 "#PWR056" H 800 2000 50  0001 C CNN
 F 1 "GND" H 800 2100 50  0000 C CNN
 F 2 "" H 800 2250 50  0001 C CNN
@@
 $EndComp
 $Comp
-L +3.3V #PWR047
+L +3.3V #PWR057
 U 1 1 59DD49A9
 P 4300 5700
-F 0 "#PWR047" H 4300 5550 50  0001 C CNN
+F 0 "#PWR057" H 4300 5550 50  0001 C CNN
 F 1 "+3.3V" H 4300 5840 50  0000 C CNN
 F 2 "" H 4300 5700 50  0001 C CNN
@@
 $EndComp
 $Comp
-L +3.3V #PWR048
+L +3.3V #PWR058
 U 1 1 59DD49E1
 P 5100 5700
-F 0 "#PWR048" H 5100 5550 50  0001 C CNN
+F 0 "#PWR058" H 5100 5550 50  0001 C CNN
 F 1 "+3.3V" H 5100 5840 50  0000 C CNN
 F 2 "" H 5100 5700 50  0001 C CNN
@@
 $EndComp
 $Comp
-L GND #PWR049
+L GND #PWR059
 U 1 1 59DD4A83
 P 4300 6800
-F 0 "#PWR049" H 4300 6550 50  0001 C CNN
+F 0 "#PWR059" H 4300 6550 50  0001 C CNN
 F 1 "GND" H 4300 6650 50  0000 C CNN
 F 2 "" H 4300 6800 50  0001 C CNN
@@
 $EndComp
 $Comp
-L GND #PWR050
+L GND #PWR060
 U 1 1 59DD4ABB
 P 5100 6800
-F 0 "#PWR050" H 5100 6550 50  0001 C CNN
+F 0 "#PWR060" H 5100 6550 50  0001 C CNN
 F 1 "GND" H 5100 6650 50  0000 C CNN
 F 2 "" H 5100 6800 50  0001 C CNN
@@
 NoConn ~ 2600 6200
 NoConn ~ 1500 2000
+Text GLabel 7000 6150 2    51   Output ~ 0
+USB_PWR_EN
+Text GLabel 7000 6250 2    51   Input ~ 0
+USB_PWR_FAULT
+Text GLabel 10200 2700 2    51   Output ~ 0
+USB_DM
+Text GLabel 10200 2800 2    51   Output ~ 0
+USB_DP
+Wire Wire Line
+	10100 2700 10200 2700
+Wire Wire Line
+	10100 2800 10200 2800
 $EndSCHEMATC

Commit message: work in progress
Parts:
- added C505, C506, C507, C508, C510: 100n, Capacitors_SMD:C_0603, symbol C
- added C509: 1u, Capacitors_SMD:C_0603, symbol C
- C501, C502: MFN (none) -> TDK; MFP (none) -> C2012X5R1A225K085AA
- C503, C504: MFN (none) -> Murata; MFP (none) -> GRM1885C1H180JA01J
- R501, R502: MFN (none) -> Panasonic; MFP (none) -> ERJ-3EKF1002V
Connections:
- net +3.3VA: now also C509.1, C510.1
- net +3V3: now also C505.1, C506.1, C507.1, C508.1
- net GND: now also C505.2, C506.2, C507.2, C508.2, C509.2, C510.2
Other:
- moved on the sheet: C503, C504, J501, J502, R501, R502, SW501, SW502, Y501

Commit message: more work
Parts:
- C505, C506, C507, C508, C510: MFN (none) -> Murata; MFP (none) -> GRM188R71E104JA01J
Changed lines of the file:
@@
+	1    0    0    -1
+$EndComp
+$Comp
+L C C505
+U 1 1 59E34530
+P 2600 7150
+F 0 "C505" H 2625 7250 50  0000 L CNN
+F 1 "100n" H 2625 7050 50  0000 L CNN
+F 2 "Capacitors_SMD:C_0603" H 2638 7000 50  0001 C CNN
+F 3 "http://datasheet.octopart.com/GRM188R71E104JA01J-Murata-datasheet-66077098.pdf" H 2600 7150 50  0001 C CNN
+F 4 "Murata" H 2625 7350 50  0001 C CNN "MFN"
+F 5 "GRM188R71E104JA01J" H 2625 7350 50  0001 C CNN "MFP"
+	1    2600 7150
+	1    0    0    -1
+$EndComp
+$Comp
+L C C506
+U 1 1 59E345BC
+P 2900 7150
+F 0 "C506" H 2925 7250 50  0000 L CNN
+F 1 "100n" H 2925 7050 50  0000 L CNN
+F 2 "Capacitors_SMD:C_0603" H 2938 7000 50  0001 C CNN
+F 3 "http://datasheet.octopart.com/GRM188R71E104JA01J-Murata-datasheet-66077098.pdf" H 2900 7150 50  0001 C CNN
+F 4 "Murata" H 2925 7350 50  0001 C CNN "MFN"
+F 5 "GRM188R71E104JA01J" H 2925 7350 50  0001 C CNN "MFP"
+	1    2900 7150
+	1    0    0    -1
+$EndComp
+$Comp
+L C C507
+U 1 1 59E34607
+P 3200 7150
+F 0 "C507" H 3225 7250 50  0000 L CNN
+F 1 "100n" H 3225 7050 50  0000 L CNN
+F 2 "Capacitors_SMD:C_0603" H 3238 7000 50  0001 C CNN
+F 3 "http://datasheet.octopart.com/GRM188R71E104JA01J-Murata-datasheet-66077098.pdf" H 3200 7150 50  0001 C CNN
+F 4 "Murata" H 3225 7350 50  0001 C CNN "MFN"
+F 5 "GRM188R71E104JA01J" H 3225 7350 50  0001 C CNN "MFP"
+	1    3200 7150
+	1    0    0    -1
+$EndComp
+$Comp
+L C C508
+U 1 1 59E34648
+P 3500 7150
+F 0 "C508" H 3525 7250 50  0000 L CNN
+F 1 "100n" H 3525 7050 50  0000 L CNN
+F 2 "Capacitors_SMD:C_0603" H 3538 7000 50  0001 C CNN
+F 3 "http://datasheet.octopart.com/GRM188R71E104JA01J-Murata-datasheet-66077098.pdf" H 3500 7150 50  0001 C CNN
+F 4 "Murata" H 3525 7350 50  0001 C CNN "MFN"
+F 5 "GRM188R71E104JA01J" H 3525 7350 50  0001 C CNN "MFP"
+	1    3500 7150
+	1    0    0    -1
+$EndComp
+$Comp
+L +3.3V #PWR061
+U 1 1 59E34B90
+P 2500 6800
+F 0 "#PWR061" H 2500 6650 50  0001 C CNN
+F 1 "+3.3V" H 2500 6940 50  0000 C CNN
+F 2 "" H 2500 6800 50  0001 C CNN
+F 3 "" H 2500 6800 50  0001 C CNN
+	1    2500 6800
+	1    0    0    -1
+$EndComp
+$Comp
+L GND #PWR062
+U 1 1 59E34BD4
+P 2500 7500
+F 0 "#PWR062" H 2500 7250 50  0001 C CNN
+F 1 "GND" H 2500 7350 50  0000 C CNN
+F 2 "" H 2500 7500 50  0001 C CNN
+F 3 "" H 2500 7500 50  0001 C CNN
+	1    2500 7500
+	1    0    0    -1
+$EndComp
+$Comp
+L +3.3VA #PWR063
+U 1 1 59E35078
+P 3900 6800
+F 0 "#PWR063" H 3900 6650 50  0001 C CNN
+F 1 "+3.3VA" H 3900 6940 50  0000 C CNN
+F 2 "" H 3900 6800 50  0001 C CNN
+F 3 "" H 3900 6800 50  0001 C CNN
+	1    3900 6800
+	1    0    0    -1
+$EndComp
+$Comp
+L GND #PWR064
+U 1 1 59E350BC
+P 3900 7500
+F 0 "#PWR064" H 3900 7250 50  0001 C CNN
+F 1 "GND" H 3900 7350 50  0000 C CNN
+F 2 "" H 3900 7500 50  0001 C CNN
+F 3 "" H 3900 7500 50  0001 C CNN
+	1    3900 7500
+	1    0    0    -1
+$EndComp
+$Comp
+L C C509
+U 1 1 59E35219
+P 4000 7150
+F 0 "C509" H 4025 7250 50  0000 L CNN
+F 1 "1u" H 4025 7050 50  0000 L CNN
+F 2 "Capacitors_SMD:C_0603" H 4038 7000 50  0001 C CNN
+F 3 "" H 4000 7150 50  0001 C CNN
+	1    4000 7150
+	1    0    0    -1
+$EndComp
+$Comp
+L C C510
+U 1 1 59E3526B
+P 4300 7150
+F 0 "C510" H 4325 7250 50  0000 L CNN
+F 1 "100n" H 4325 7050 50  0000 L CNN
+F 2 "Capacitors_SMD:C_0603" H 4338 7000 50  0001 C CNN
+F 3 "http://datasheet.octopart.com/GRM188R71E104JA01J-Murata-datasheet-66077098.pdf" H 4300 7150 50  0001 C CNN
+F 4 "Murata" H 4325 7350 50  0001 C CNN "MFN"
+F 5 "GRM188R71E104JA01J" H 4325 7350 50  0001 C CNN "MFP"
+	1    4300 7150
 	1    0    0    -1
 $EndComp
@@
 Wire Wire Line
 	10100 2800 10200 2800
+Wire Wire Line
+	2500 6900 3500 6900
+Wire Wire Line
+	2600 6900 2600 7000
+Wire Wire Line
+	2900 6900 2900 7000
+Wire Wire Line
+	3200 6900 3200 7000
+Wire Wire Line
+	3500 6900 3500 7000
+Wire Wire Line
+	2500 6900 2500 6800
+Wire Wire Line
+	2500 7400 3500 7400
+Wire Wire Line
+	2600 7400 2600 7300
+Wire Wire Line
+	2900 7400 2900 7300
+Wire Wire Line
+	3500 7400 3500 7300
+Wire Wire Line
+	3200 7300 3200 7400
+Wire Wire Line
+	2500 7400 2500 7500
+Wire Wire Line
+	3900 7500 3900 7400
+Wire Wire Line
+	3900 7400 4300 7400
+Wire Wire Line
+	4000 7400 4000 7300
+Wire Wire Line
+	3900 6800 3900 6900
+Wire Wire Line
+	3900 6900 4300 6900
+Wire Wire Line
+	4000 6900 4000 7000
+Wire Wire Line
+	4300 6900 4300 7000
+Wire Wire Line
+	4300 7400 4300 7300
 Connection ~ 2500 6000
 Connection ~ 2500 5800
@@
 Connection ~ 5900 6800
 Connection ~ 6500 6900
+Connection ~ 2600 6900
+Connection ~ 2900 6900
+Connection ~ 3200 6900
+Connection ~ 2600 7400
+Connection ~ 2900 7400
+Connection ~ 3200 7400
+Connection ~ 4000 6900
+Connection ~ 4000 7400
 NoConn ~ 1500 5600
 NoConn ~ 1500 5900
@@
 NoConn ~ 2600 5900
 NoConn ~ 1500 2000
-$Comp
-L C C505
-U 1 1 59E34530
-P 2600 7150
-F 0 "C505" H 2625 7250 50  0000 L CNN
-F 1 "100n" H 2625 7050 50  0000 L CNN
-F 2 "Capacitors_SMD:C_0603" H 2638 7000 50  0001 C CNN
-F 3 "" H 2600 7150 50  0001 C CNN
-	1    2600 7150
-	1    0    0    -1
-$EndComp
-$Comp
-L C C506
-U 1 1 59E345BC
-P 2900 7150
-F 0 "C506" H 2925 7250 50  0000 L CNN
-F 1 "100n" H 2925 7050 50  0000 L CNN
-F 2 "Capacitors_SMD:C_0603" H 2938 7000 50  0001 C CNN
-F 3 "" H 2900 7150 50  0001 C CNN
-	1    2900 7150
-	1    0    0    -1
-$EndComp
-$Comp
-L C C507
-U 1 1 59E34607
-P 3200 7150
-F 0 "C507" H 3225 7250 50  0000 L CNN
-F 1 "100n" H 3225 7050 50  0000 L CNN
-F 2 "Capacitors_SMD:C_0603" H 3238 7000 50  0001 C CNN
-F 3 "" H 3200 7150 50  0001 C CNN
-	1    3200 7150
-	1    0    0    -1
-$EndComp
-$Comp
-L C C508
-U 1 1 59E34648
-P 3500 7150
-F 0 "C508" H 3525 7250 50  0000 L CNN
-F 1 "100n" H 3525 7050 50  0000 L CNN
-F 2 "Capacitors_SMD:C_0603" H 3538 7000 50  0001 C CNN
-F 3 "" H 3500 7150 50  0001 C CNN
-	1    3500 7150
-	1    0    0    -1
-$EndComp
-Wire Wire Line
-	2500 6900 3500 6900
-Wire Wire Line
-	2600 6900 2600 7000
-Wire Wire Line
-	2900 6900 2900 7000
-Connection ~ 2600 6900
-Wire Wire Line
-	3200 6900 3200 7000
-Connection ~ 2900 6900
-Wire Wire Line
-	3500 6900 3500 7000
-Connection ~ 3200 6900
-Wire Wire Line
-	2500 6900 2500 6800
-Wire Wire Line
-	2500 7400 3500 7400
-Wire Wire Line
-	2600 7400 2600 7300
-Wire Wire Line
-	2900 7400 2900 7300
-Connection ~ 2600 7400
-Wire Wire Line
-	3500 7400 3500 7300
-Connection ~ 2900 7400
-Wire Wire Line
-	3200 7300 3200 7400
-Connection ~ 3200 7400
-Wire Wire Line
-	2500 7400 2500 7500
-$Comp
-L +3.3V #PWR061
-U 1 1 59E34B90
-P 2500 6800
-F 0 "#PWR061" H 2500 6650 50  0001 C CNN
-F 1 "+3.3V" H 2500 6940 50  0000 C CNN
-F 2 "" H 2500 6800 50  0001 C CNN
-F 3 "" H 2500 6800 50  0001 C CNN
-	1    2500 6800
-	1    0    0    -1
-$EndComp
-$Comp
-L GND #PWR062
-U 1 1 59E34BD4
-P 2500 7500
-F 0 "#PWR062" H 2500 7250 50  0001 C CNN
-F 1 "GND" H 2500 7350 50  0000 C CNN
-F 2 "" H 2500 7500 50  0001 C CNN
-F 3 "" H 2500 7500 50  0001 C CNN
-	1    2500 7500
-	1    0    0    -1
-$EndComp
-$Comp
-L +3.3VA #PWR063
-U 1 1 59E35078
-P 3900 6800
-F 0 "#PWR063" H 3900 6650 50  0001 C CNN
-F 1 "+3.3VA" H 3900 6940 50  0000 C CNN
-F 2 "" H 3900 6800 50  0001 C CNN
-F 3 "" H 3900 6800 50  0001 C CNN
-	1    3900 6800
-	1    0    0    -1
-$EndComp
-$Comp
-L GND #PWR064
-U 1 1 59E350BC
-P 3900 7500
-F 0 "#PWR064" H 3900 7250 50  0001 C CNN
-F 1 "GND" H 3900 7350 50  0000 C CNN
-F 2 "" H 3900 7500 50  0001 C CNN
-F 3 "" H 3900 7500 50  0001 C CNN
-	1    3900 7500
-	1    0    0    -1
-$EndComp
-Wire Wire Line
-	3900 7500 3900 7400
-Wire Wire Line
-	3900 7400 4300 7400
-Wire Wire Line
-	4000 7400 4000 7300
-Wire Wire Line
-	3900 6800 3900 6900
-Wire Wire Line
-	3900 6900 4300 6900
-Wire Wire Line
-	4000 6900 4000 7000
-$Comp
-L C C509
-U 1 1 59E35219
-P 4000 7150
-F 0 "C509" H 4025 7250 50  0000 L CNN
-F 1 "1u" H 4025 7050 50  0000 L CNN
-F 2 "Capacitors_SMD:C_0603" H 4038 7000 50  0001 C CNN
-F 3 "" H 4000 7150 50  0001 C CNN
-	1    4000 7150
-	1    0    0    -1
-$EndComp
-$Comp
-L C C510
-U 1 1 59E3526B
-P 4300 7150
-F 0 "C510" H 4325 7250 50  0000 L CNN
-F 1 "100n" H 4325 7050 50  0000 L CNN
-F 2 "Capacitors_SMD:C_0603" H 4338 7000 50  0001 C CNN
-F 3 "" H 4300 7150 50  0001 C CNN
-	1    4300 7150
-	1    0    0    -1
-$EndComp
-Wire Wire Line
-	4300 6900 4300 7000
-Connection ~ 4000 6900
-Wire Wire Line
-	4300 7400 4300 7300
-Connection ~ 4000 7400
 $EndSCHEMATC

Commit message: more work on layout
Connections:
- net SPI1_MISO is gone; now on net SR_MISO: U501.22 (ADC1_IN6/ADC2_IN6/SPI1_MISO/TIM13_CH1/TIM1_BKIN/TIM3_CH1/TIM8_BKIN/PA6)
- net SPI1_MOSI is gone; now on net SR_MOSI: U501.23 (ADC1_IN7/ADC2_IN7/SPI1_MOSI/TIM14_CH1/TIM1_CH1N/TIM3_CH2/TIM8_CH1N/PA7)
- net SPI1_SCK is gone; now on net SR_SCK: U501.21 (ADC1_IN5/ADC2_IN5/DAC_OUT2/SPI1_SCK/TIM2_CH1/TIM2_ETR/TIM8_CH1N/USB_OTG_HS_ULPI_CK/PA5)
- net DAC_MOSI: now also U501.57 (CAN2_RX/I2C1_SMBA/I2S3_SD/SPI1_MOSI/SPI3_MOSI/TIM3_CH2/USB_OTG_HS_ULPI_D7/PB5)
- net DAC_SCK: now also U501.51 (PC10/I2S3_CK/SDIO_D2/SPI3_SCK/UART4_TX/USART3_TX)
- net LCD_CS: now also U501.33 (CAN2_RX/I2C2_SMBA/I2S2_WS/SPI2_NSS/TIM1_BKIN/USART3_CK/USB_OTG_HS_ID/USB_OTG_HS_ULPI_D5/PB12)
- net LCD_DC: now also U501.36 (ADC1_EXTI15/ADC2_EXTI15/ADC3_EXTI15/I2S2_SD/RTC_REFIN/SPI2_MOSI/TIM12_CH2/TIM1_CH3N/TIM8_CH3N/USB_OTG_HS_DP/PB15)
- net LCD_MOSI: now also U501.11 (PC3/ADC1_IN13/ADC2_IN13/ADC3_IN13/I2S2_SD/SPI2_MOSI/USB_OTG_HS_ULPI_NXT)
- net LCD_RES: now also U501.35 (I2S2_ext_SD/SPI2_MISO/TIM12_CH1/TIM1_CH2N/TIM8_CH2N/USART3_RTS/USB_OTG_HS_DM/PB14)
- net LCD_SCK: now also U501.34 (CAN2_TX/I2S2_CK/SPI2_SCK/TIM1_CH1N/USART3_CTS/USB_OTG_HS_ULPI_D6/USB_OTG_HS_VBUS/PB13)
- net SPI2_MOSI: no longer U501.11 (PC3/ADC1_IN13/ADC2_IN13/ADC3_IN13/I2S2_SD/SPI2_MOSI/USB_OTG_HS_ULPI_NXT)
- net SPI2_SCK: no longer U501.34 (CAN2_TX/I2S2_CK/SPI2_SCK/TIM1_CH1N/USART3_CTS/USB_OTG_HS_ULPI_D6/USB_OTG_HS_VBUS/PB13)
- net SPI3_MOSI: no longer U501.57 (CAN2_RX/I2C1_SMBA/I2S3_SD/SPI1_MOSI/SPI3_MOSI/TIM3_CH2/USB_OTG_HS_ULPI_D7/PB5)
- net SPI3_SCK: no longer U501.51 (PC10/I2S3_CK/SDIO_D2/SPI3_SCK/UART4_TX/USART3_TX)
- net SR_LATCH: now also U501.26 (ADC1_IN8/ADC2_IN8/TIM1_CH2N/TIM3_CH3/TIM8_CH2N/USB_OTG_HS_ULPI_D1/PB0)
- net SR_LOAD: now also U501.27 (ADC1_IN9/ADC2_IN9/TIM1_CH3N/TIM3_CH4/TIM8_CH3N/USB_OTG_HS_ULPI_D2/PB1)
- net USB_DM renamed USB_D-
- net USB_DP renamed USB_D+
Changed lines of the file:
@@
 Text GLabel 1400 4000 0    51   Input ~ 0
 MIDI_RX
-Text GLabel 8400 5600 2    51   Output ~ 0
+Text GLabel 1400 3600 0    51   Output ~ 0
 LCD_MOSI
-Text GLabel 8400 5700 2    51   Output ~ 0
+Text GLabel 10200 4600 2    51   Output ~ 0
 LCD_SCK
-Text GLabel 8400 5800 2    51   Output ~ 0
+Text GLabel 10200 4500 2    51   Output ~ 0
 LCD_CS
-Text GLabel 8400 5900 2    51   Output ~ 0
+Text GLabel 10200 4700 2    51   Output ~ 0
 LCD_RES
-Text GLabel 8400 6000 2    51   Output ~ 0
+Text GLabel 10200 4800 2    51   Output ~ 0
 LCD_DC
 Text GLabel 1400 4600 0    51   Input ~ 0
@@
 Text GLabel 1400 4800 0    51   Input ~ 0
 ENC_SW
-Text GLabel 10200 2100 2    51   Output ~ 0
-SPI1_SCK
-Text GLabel 10200 2200 2    51   Input ~ 0
-SPI1_MISO
-Text GLabel 10200 2300 2    51   Output ~ 0
-SPI1_MOSI
 Text GLabel 1400 3500 0    51   Input ~ 0
 SPI2_MISO
-Text GLabel 1400 3600 0    51   Output ~ 0
+Text GLabel 900  3600 0    51   Output ~ 0
 SPI2_MOSI
-Text GLabel 10200 4600 2    51   Output ~ 0
+Text GLabel 10700 4600 2    51   Output ~ 0
 SPI2_SCK
-Text GLabel 10200 3800 2    51   Output ~ 0
+Text GLabel 10700 3800 2    51   Output ~ 0
 SPI3_MOSI
-Text GLabel 1400 4300 0    51   Output ~ 0
+Text GLabel 900  4300 0    51   Output ~ 0
 SPI3_SCK
 Text GLabel 1400 4400 0    51   Input ~ 0
@@
 Text GLabel 7000 5900 2    51   Input ~ 0
 RES_IN
-Text GLabel 9400 5500 2    51   Output ~ 0
+Text GLabel 10200 2300 2    51   Output ~ 0
 SR_MOSI
-Text GLabel 9400 5600 2    51   Output ~ 0
+Text GLabel 10200 2200 2    51   Input ~ 0
 SR_MISO
-Text GLabel 9400 5700 2    51   Output ~ 0
+Text GLabel 10200 2100 2    51   Output ~ 0
 SR_SCK
-Text GLabel 9400 5800 2    51   Output ~ 0
+Text GLabel 10200 3300 2    51   Output ~ 0
 SR_LATCH
-Text GLabel 9400 5900 2    51   Output ~ 0
+Text GLabel 10200 3400 2    51   Output ~ 0
 SR_LOAD
-Text GLabel 9400 6200 2    51   Output ~ 0
+Text GLabel 10200 3800 2    51   Output ~ 0
 DAC_MOSI
-Text GLabel 9400 6300 2    51   Output ~ 0
+Text GLabel 1400 4300 0    51   Output ~ 0
 DAC_SCK
-Text GLabel 7000 6150 2    51   Output ~ 0
+Text GLabel 7800 5600 2    51   Output ~ 0
 USB_PWR_EN
-Text GLabel 7000 6250 2    51   Input ~ 0
+Text GLabel 7800 5700 2    51   Input ~ 0
 USB_PWR_FAULT
 Text GLabel 10200 2700 2    51   Output ~ 0
-USB_DM
+USB_D-
 Text GLabel 10200 2800 2    51   Output ~ 0
-USB_DP
+USB_D+
 Wire Wire Line
 	1500 6100 1600 6100
@@
 NoConn ~ 2600 5900
 NoConn ~ 1500 2000
+Wire Wire Line
+	10100 3300 10200 3300
+Wire Wire Line
+	10100 3400 10200 3400
+Wire Wire Line
+	10100 4500 10200 4500
+Wire Wire Line
+	10100 4700 10200 4700
+Wire Wire Line
+	10100 4800 10200 4800
 $EndSCHEMATC
