File: dac.sch (KiCad schematic (older format))
At the start: 1 part, among them U701 DAC8568C

Commit message: work on schematic
Connections:
- net +3V3: now reaches U701.3 (AVDD)
- net AREF_2.048V: now reaches U701.8 (VREF)
Changed lines of the file:
@@
 EESchema Schematic File Version 2
+LIBS:w_power
 LIBS:w_lcd
 LIBS:w_stm32
@@
 encoding utf-8
 Sheet 7 7
-Title ""
+Title "Eurorack Sequencer"
 Date ""
-Rev ""
-Comp ""
+Rev "0.1"
+Comp "westlicht"
 Comment1 ""
 Comment2 ""
@@
 $EndComp
 $Comp
-L GND #PWR099
+L GND #PWR0109
 U 1 1 59DDC913
 P 1400 3200
-F 0 "#PWR099" H 1400 2950 50  0001 C CNN
+F 0 "#PWR0109" H 1400 2950 50  0001 C CNN
 F 1 "GND" H 1400 3050 50  0000 C CNN
 F 2 "" H 1400 3200 50  0001 C CNN
@@
 Wire Wire Line
 	1400 3000 1500 3000
+Wire Wire Line
+	1400 2300 1400 2400
+Wire Wire Line
+	1400 2400 1500 2400
+Wire Wire Line
+	1500 2500 1400 2500
+Text GLabel 1400 2500 0    51   Input ~ 0
+AREF_2.048V
+$Comp
+L +3.3V #PWR0110
+U 1 1 59E0CF3B
+P 1400 2300
+F 0 "#PWR0110" H 1400 2150 50  0001 C CNN
+F 1 "+3.3V" H 1400 2440 50  0000 C CNN
+F 2 "" H 1400 2300 50  0001 C CNN
+F 3 "" H 1400 2300 50  0001 C CNN
+	1    1400 2300
+	1    0    0    -1
+$EndComp
 $EndSCHEMATC

Commit message: work in progress
Parts:
- added C701, C702, C703, C704, C705, C706, C707, C708: 18p, Capacitors_SMD:C_0603, symbol C
- added C709, C710, C711, C712: 100n, Capacitors_SMD:C_0603, symbol C
- added R701, R702, R703, R704, R713, R714, R715, R716: 220, Resistors_SMD:R_0603, symbol R
- added R705, R707, R709, R711, R717, R719, R721, R723: 24.9k, Resistors_SMD:R_0603, symbol R
- added R706, R708, R710, R712, R718, R720, R722, R724: 75k, Resistors_SMD:R_0603, symbol R
- added U702, U703: OPA4172, Housings_SOIC:SOIC-14_3.9x8.7mm_Pitch1.27mm, symbol OPA4134
Connections:
- net DAC1: now also U702.3 (+)
- net DAC2: now also U702.5 (+)
- net DAC3: now also U702.10 (+)
- net DAC4: now also U702.12 (+)
- net DAC5: now also U703.3 (+)
- net DAC6: now also U703.5 (+)
- net DAC7: now also U703.10 (+)
- net DAC8: now also U703.12 (+)
- net GND: now also C709.2, C710.2, C711.1, C712.1, R705.2, R707.2, R709.2, R711.2, R717.2, R719.2, R721.2, R723.2
- new net: C702.2, R707.1, R708.2, U702.6 (-)
- new net: R702.2, U702.7
- new net: C704.2, R711.1, R712.2, U702.13 (-)
- new net: R704.2, U702.14
- new net: C706.2, R719.1, R720.2, U703.6 (-)
- new net: R714.2, U703.7
- new net: R701.2, U702.1
- new net: C701.2, R705.1, R706.2, U702.2 (-)
- new net: R703.2, U702.8
- new net: C703.2, R709.1, R710.2, U702.9 (-)
- new net: R713.2, U703.1
- new net: C705.2, R717.1, R718.2, U703.2 (-)
- new net: R715.2, U703.8
- new net: C707.2, R721.1, R722.2, U703.9 (-)
- new net: C708.2, R723.1, R724.2, U703.13 (-)
- new net: R716.2, U703.14
- new net +12V: C709.1, C710.1, U702.4 (V+), U702.4 (V+), U702.4 (V+), U702.4 (V+), U703.4 (V+), U703.4 (V+), U703.4 (V+), U703.4 (V+)
- new net -12V: C711.2, C712.2, U702.11 (V-), U702.11 (V-), U702.11 (V-), U702.11 (V-), U703.11 (V-), U703.11 (V-), U703.11 (V-), U703.11 (V-)
- new net CV1: C701.1, R701.1, R706.1
- new net CV2: C702.1, R702.1, R708.1
- new net CV3: C703.1, R703.1, R710.1
- new net CV4: C704.1, R704.1, R712.1
- new net CV5: C705.1, R713.1, R718.1
- new net CV6: C706.1, R714.1, R720.1
- new net CV7: C707.1, R715.1, R722.1
- new net CV8: C708.1, R716.1, R724.1

Commit message: more work
Parts:
- C701, C702, C703, C704, C705, C706, C707, C708: MFN (none) -> Murata; MFP (none) -> GRM1885C1H180JA01J
- C709, C710, C711, C712: MFN (none) -> Murata; MFP (none) -> GRM188R71E104JA01J
- U702, U703: MFN (none) -> Texas Instruments; MFP (none) -> OPA4172IPW

Commit message: more work on layout
Parts:
- added C713, C716: 2.2u, Capacitors_SMD:C_0805, symbol C
- added C714, C715: 100n, Capacitors_SMD:C_0603, symbol C
Connections:
- net AREF_2.048V: now also C713.1, C714.1
- net GND: now also C713.2, C714.2, C715.2, C716.2
- net +3V3 renamed +3.3VA
- net +3.3VA: now also C715.1, C716.1
Other:
- moved on the sheet: C701, C702, C703, C704, C705, C706, C707, C708, C709, C710, C711, C712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

Commit message: redesign in progress
Parts:
- added C717: 100n, Capacitors_SMD:C_0603, symbol C
- added R725: 33k, Resistors_SMD:R_0603, symbol R
- added R726: 22k, Resistors_SMD:R_0603, symbol R
- R705, R707, R709, R711, R717, R719, R721, R723: value 24.9k -> 24k; MFP ERJ-3EKF2492V -> ERJ-3EKF2402V
- R706, R708, R710, R712, R718, R720, R722, R724: value 75k -> 100k; MFP ERJ-3EKF7502V -> ERJ-3EKF1003V
Connections:
- net DAC1: now also R705.2; no longer U702.3 (+)
- net DAC2: now also R707.2; no longer U702.5 (+)
- net DAC3: now also R709.2; no longer U702.10 (+)
- net DAC4: now also R711.2; no longer U702.12 (+)
- net DAC5: now also R717.2; no longer U703.3 (+)
- net DAC6: now also R719.2; no longer U703.5 (+)
- net DAC7: now also R721.2; no longer U703.10 (+)
- net DAC8: now also R723.2; no longer U703.12 (+)
- net GND: now also C717.2, R726.2; no longer R705.2, R707.2, R709.2, R711.2, R717.2, R719.2, R721.2, R723.2
- net AREF_2.048V: no longer names the net of C713.1, C714.1, U701.8 (VREF)
- net AREF_2.048V: now also R725.1
- new net VBIAS: C717.1, R725.2, R726.1, U702.10 (+), U702.12 (+), U702.3 (+), U702.5 (+), U703.10 (+), U703.12 (+), U703.3 (+), U703.5 (+)
Other:
- moved on the sheet: C701, C702, C704, C705, C706, C708, C713, C714, R701, R702, R704, R705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

Commit message: only ground plane left
Connections:
- net +3.3VA: now also U701.9 (~CLR)
- net GND: now also U701.1 (~LDAC)
- net DAC_SYNC: now reaches U701.2 (~SYNC)
Changed lines of the file:
@@
 $EndComp
 $Comp
-L GND #PWR723
+L GND #PWR0114
 U 1 1 59DDC913
-P 3900 6100
-F 0 "#PWR723" H 3900 5850 50  0001 C CNN
-F 1 "GND" H 3900 5950 50  0000 C CNN
-F 2 "" H 3900 6100 50  0001 C CNN
-F 3 "" H 3900 6100 50  0001 C CNN
-	1    3900 6100
+P 3800 6100
+F 0 "#PWR0114" H 3800 5850 50  0001 C CNN
+F 1 "GND" H 3800 5950 50  0000 C CNN
+F 2 "" H 3800 6100 50  0001 C CNN
+F 3 "" H 3800 6100 50  0001 C CNN
+	1    3800 6100
 	1    0    0    -1
 $EndComp
@@
 $EndComp
 $Comp
-L +12V #PWR701
+L +12V #PWR0115
 U 1 1 59E02DC5
 P 2500 1200
-F 0 "#PWR701" H 2500 1050 50  0001 C CNN
+F 0 "#PWR0115" H 2500 1050 50  0001 C CNN
 F 1 "+12V" H 2500 1340 50  0000 C CNN
 F 2 "" H 2500 1200 50  0001 C CNN
@@
 $EndComp
 $Comp
-L -12V #PWR705
+L -12V #PWR707
 U 1 1 59E373B3
 P 2500 1800
-F 0 "#PWR705" H 2500 1900 50  0001 C CNN
+F 0 "#PWR707" H 2500 1900 50  0001 C CNN
 F 1 "-12V" H 2500 1950 50  0000 C CNN
 F 2 "" H 2500 1800 50  0001 C CNN
@@
 $EndComp
 $Comp
-L +12V #PWR702
+L +12V #PWR0116
 U 1 1 59E399A0
 P 4700 1200
-F 0 "#PWR702" H 4700 1050 50  0001 C CNN
+F 0 "#PWR0116" H 4700 1050 50  0001 C CNN
 F 1 "+12V" H 4700 1340 50  0000 C CNN
 F 2 "" H 4700 1200 50  0001 C CNN
@@
 $EndComp
 $Comp
-L -12V #PWR706
+L -12V #PWR708
 U 1 1 59E399CD
 P 4700 1800
-F 0 "#PWR706" H 4700 1900 50  0001 C CNN
+F 0 "#PWR708" H 4700 1900 50  0001 C CNN
 F 1 "-12V" H 4700 1950 50  0000 C CNN
 F 2 "" H 4700 1800 50  0001 C CNN
@@
 $EndComp
 $Comp
-L +12V #PWR703
+L +12V #PWR0117
 U 1 1 59E39C85
 P 6900 1200
-F 0 "#PWR703" H 6900 1050 50  0001 C CNN
+F 0 "#PWR0117" H 6900 1050 50  0001 C CNN
 F 1 "+12V" H 6900 1340 50  0000 C CNN
 F 2 "" H 6900 1200 50  0001 C CNN
@@
 $EndComp
 $Comp
-L -12V #PWR707
+L -12V #PWR709
 U 1 1 59E39CB2
 P 6900 1800
-F 0 "#PWR707" H 6900 1900 50  0001 C CNN
+F 0 "#PWR709" H 6900 1900 50  0001 C CNN
 F 1 "-12V" H 6900 1950 50  0000 C CNN
 F 2 "" H 6900 1800 50  0001 C CNN
@@
 $EndComp
 $Comp
-L +12V #PWR704
+L +12V #PWR0118
 U 1 1 59E39CCE
 P 9100 1200
-F 0 "#PWR704" H 9100 1050 50  0001 C CNN
+F 0 "#PWR0118" H 9100 1050 50  0001 C CNN
 F 1 "+12V" H 9100 1340 50  0000 C CNN
 F 2 "" H 9100 1200 50  0001 C CNN
@@
 $EndComp
 $Comp
-L -12V #PWR708
+L -12V #PWR710
 U 1 1 59E39CFB
 P 9100 1800
-F 0 "#PWR708" H 9100 1900 50  0001 C CNN
+F 0 "#PWR710" H 9100 1900 50  0001 C CNN
 F 1 "-12V" H 9100 1950 50  0000 C CNN
 F 2 "" H 9100 1800 50  0001 C CNN
@@
 $EndComp
 $Comp
-L +12V #PWR709
+L +12V #PWR0119
 U 1 1 59E3B294
 P 2500 2900
-F 0 "#PWR709" H 2500 2750 50  0001 C CNN
+F 0 "#PWR0119" H 2500 2750 50  0001 C CNN
 F 1 "+12V" H 2500 3040 50  0000 C CNN
 F 2 "" H 2500 2900 50  0001 C CNN
@@
 $EndComp
 $Comp
-L -12V #PWR713
+L -12V #PWR715
 U 1 1 59E3B2C1
 P 2500 3500
-F 0 "#PWR713" H 2500 3600 50  0001 C CNN
+F 0 "#PWR715" H 2500 3600 50  0001 C CNN
 F 1 "-12V" H 2500 3650 50  0000 C CNN
 F 2 "" H 2500 3500 50  0001 C CNN
@@
 $EndComp
 $Comp
-L +12V #PWR710
+L +12V #PWR0120
 U 1 1 59E3B2D9
 P 4700 2900
-F 0 "#PWR710" H 4700 2750 50  0001 C CNN
+F 0 "#PWR0120" H 4700 2750 50  0001 C CNN
 F 1 "+12V" H 4700 3040 50  0000 C CNN
 F 2 "" H 4700 2900 50  0001 C CNN
@@
 $EndComp
 $Comp
-L -12V #PWR714
+L -12V #PWR716
 U 1 1 59E3B306
 P 4700 3500
-F 0 "#PWR714" H 4700 3600 50  0001 C CNN
+F 0 "#PWR716" H 4700 3600 50  0001 C CNN
 F 1 "-12V" H 4700 3650 50  0000 C CNN
 F 2 "" H 4700 3500 50  0001 C CNN
@@
 $EndComp
 $Comp
-L +12V #PWR711
+L +12V #PWR0121
 U 1 1 59E3B31E
 P 6900 2900
-F 0 "#PWR711" H 6900 2750 50  0001 C CNN
+F 0 "#PWR0121" H 6900 2750 50  0001 C CNN
 F 1 "+12V" H 6900 3040 50  0000 C CNN
 F 2 "" H 6900 2900 50  0001 C CNN
@@
 $EndComp
 $Comp
-L -12V #PWR715
+L -12V #PWR717
 U 1 1 59E3B34B
 P 6900 3500
-F 0 "#PWR715" H 6900 3600 50  0001 C CNN
+F 0 "#PWR717" H 6900 3600 50  0001 C CNN
 F 1 "-12V" H 6900 3650 50  0000 C CNN
 F 2 "" H 6900 3500 50  0001 C CNN
@@
 $EndComp
 $Comp
-L +12V #PWR712
+L +12V #PWR0122
 U 1 1 59E3B363
 P 9100 2900
-F 0 "#PWR712" H 9100 2750 50  0001 C CNN
+F 0 "#PWR0122" H 9100 2750 50  0001 C CNN
 F 1 "+12V" H 9100 3040 50  0000 C CNN
 F 2 "" H 9100 2900 50  0001 C CNN
@@
 $EndComp
 $Comp
-L -12V #PWR716
+L -12V #PWR718
 U 1 1 59E3B390
 P 9100 3500
-F 0 "#PWR716" H 9100 3600 50  0001 C CNN
+F 0 "#PWR718" H 9100 3600 50  0001 C CNN
 F 1 "-12V" H 9100 3650 50  0000 C CNN
 F 2 "" H 9100 3500 50  0001 C CNN
@@
 $EndComp
 $Comp
-L -12V #PWR722
+L -12V #PWR724
 U 1 1 59E3CB0F
 P 7700 6000
-F 0 "#PWR722" H 7700 6100 50  0001 C CNN
+F 0 "#PWR724" H 7700 6100 50  0001 C CNN
 F 1 "-12V" H 7700 6150 50  0000 C CNN
 F 2 "" H 7700 6000 50  0001 C CNN
@@
 $EndComp
 $Comp
-L +12V #PWR717
+L +12V #PWR0123
 U 1 1 59E3CBD7
 P 7700 4800
-F 0 "#PWR717" H 7700 4650 50  0001 C CNN
+F 0 "#PWR0123" H 7700 4650 50  0001 C CNN
 F 1 "+12V" H 7700 4940 50  0000 C CNN
 F 2 "" H 7700 4800 50  0001 C CNN
@@
 $EndComp
 $Comp
-L GND #PWR720
+L GND #PWR0124
 U 1 1 59E3CC72
 P 7600 5500
-F 0 "#PWR720" H 7600 5250 50  0001 C CNN
+F 0 "#PWR0124" H 7600 5250 50  0001 C CNN
 F 1 "GND" H 7600 5350 50  0000 C CNN
 F 2 "" H 7600 5500 50  0001 C CNN
@@
 $EndComp
 $Comp
-L +3.3VA #PWR719
+L +3.3VA #PWR0125
 U 1 1 59E85A18
 P 6500 5300
-F 0 "#PWR719" H 6500 5150 50  0001 C CNN
+F 0 "#PWR0125" H 6500 5150 50  0001 C CNN
 F 1 "+3.3VA" H 6500 5440 50  0000 C CNN
 F 2 "" H 6500 5300 50  0001 C CNN
@@
 $EndComp
 $Comp
-L GND #PWR721
+L GND #PWR0126
 U 1 1 59E85AB9
 P 6500 6000
-F 0 "#PWR721" H 6500 5750 50  0001 C CNN
+F 0 "#PWR0126" H 6500 5750 50  0001 C CNN
 F 1 "GND" H 6500 5850 50  0000 C CNN
 F 2 "" H 6500 6000 50  0001 C CNN
@@
 $EndComp
 $Comp
-L GND #PWR726
+L GND #PWR0127
 U 1 1 59E89BC5
 P 2900 6400
-F 0 "#PWR726" H 2900 6150 50  0001 C CNN
+F 0 "#PWR0127" H 2900 6150 50  0001 C CNN
 F 1 "GND" H 2900 6250 50  0000 C CNN
 F 2 "" H 2900 6400 50  0001 C CNN
@@
 $EndComp
 $Comp
-L GND #PWR727
+L GND #PWR0128
 U 1 1 59E89C6C
 P 3200 6400
-F 0 "#PWR727" H 3200 6150 50  0001 C CNN
+F 0 "#PWR0128" H 3200 6150 50  0001 C CNN
 F 1 "GND" H 3200 6250 50  0000 C CNN
 F 2 "" H 3200 6400 50  0001 C CNN
@@
 $EndComp
 $Comp
-L +3.3VA #PWR718
+L +3.3VA #PWR0129
 U 1 1 59EA8926
 P 3900 5200
-F 0 "#PWR718" H 3900 5050 50  0001 C CNN
+F 0 "#PWR0129" H 3900 5050 50  0001 C CNN
 F 1 "+3.3VA" H 3900 5340 50  0000 C CNN
 F 2 "" H 3900 5200 50  0001 C CNN
@@
 $EndComp
 $Comp
-L GND #PWR725
+L GND #PWR0130
 U 1 1 59F01739
 P 2600 6400
-F 0 "#PWR725" H 2600 6150 50  0001 C CNN
+F 0 "#PWR0130" H 2600 6150 50  0001 C CNN
 F 1 "GND" H 2600 6250 50  0000 C CNN
 F 2 "" H 2600 6400 50  0001 C CNN
@@
 $EndComp
 $Comp
-L GND #PWR724
+L GND #PWR0131
 U 1 1 59F021DB
 P 2300 6400
-F 0 "#PWR724" H 2300 6150 50  0001 C CNN
+F 0 "#PWR0131" H 2300 6150 50  0001 C CNN
 F 1 "GND" H 2300 6250 50  0000 C CNN
 F 2 "" H 2300 6400 50  0001 C CNN
@@
 Text GLabel 5200 6000 2    51   Output ~ 0
 DAC8
-Text GLabel 3900 5900 0    51   Input ~ 0
+Text GLabel 3700 5900 0    51   Input ~ 0
 DAC_SCK
-Text GLabel 3900 5800 0    51   Input ~ 0
+Text GLabel 3700 5800 0    51   Input ~ 0
 DAC_MOSI
 Text GLabel 1700 2100 0    51   Input ~ 0
@@
 	5100 6000 5200 6000
 Wire Wire Line
-	3900 6100 3900 6000
-Wire Wire Line
-	3900 6000 4000 6000
-Wire Wire Line
-	3900 5800 4000 5800
-Wire Wire Line
-	3900 5900 4000 5900
-Wire Wire Line
-	3900 5200 3900 5300
+	3800 6000 4000 6000
+Wire Wire Line
+	3700 5800 4000 5800
+Wire Wire Line
+	3700 5900 4000 5900
+Wire Wire Line
+	3900 5200 3900 5700
 Wire Wire Line
 	3900 5300 4000 5300
@@
 	2600 6400 2600 6300
 Wire Wire Line
-	2600 6000 2600 5800
+	2600 5800 2600 6000
 Wire Wire Line
 	2600 5500 2600 5400
@@
 Connection ~ 2600 5900
 Connection ~ 2300 5900
+Wire Wire Line
+	3900 5700 4000 5700
+Connection ~ 3900 5300
+Text GLabel 3700 5600 0    51   Input ~ 0
+DAC_SYNC
+Wire Wire Line
+	3700 5600 4000 5600
+Wire Wire Line
+	3800 5500 3800 6100
+Wire Wire Line
+	3800 5500 4000 5500
+Connection ~ 3800 6000
+$Comp
+L +12V #PWR0132
+U 1 1 59F3FADC
+P 900 900
+F 0 "#PWR0132" H 900 750 50  0001 C CNN
+F 1 "+12V" H 900 1040 50  0000 C CNN
+F 2 "" H 900 900 50  0001 C CNN
+F 3 "" H 900 900 50  0001 C CNN
+	1    900  900
+	1    0    0    -1
+$EndComp
+$Comp
+L -12V #PWR706
+U 1 1 59F3FE98
+P 900 1400
+F 0 "#PWR706" H 900 1500 50  0001 C CNN
+F 1 "-12V" H 900 1550 50  0000 C CNN
+F 2 "" H 900 1400 50  0001 C CNN
+F 3 "" H 900 1400 50  0001 C CNN
+	1    900  1400
+	1    0    0    -1
+$EndComp
+$Comp
+L PWR_FLAG #FLG0133
+U 1 1 59F40358
+P 900 900
+F 0 "#FLG0133" H 900 975 50  0001 C CNN
+F 1 "PWR_FLAG" H 900 1050 50  0000 C CNN
+F 2 "" H 900 900 50  0001 C CNN
+F 3 "" H 900 900 50  0001 C CNN
+	1    900  900
+	-1   0    0    1
+$EndComp
+$Comp
+L PWR_FLAG #FLG0134
+U 1 1 59F40408
+P 900 1400
+F 0 "#FLG0134" H 900 1475 50  0001 C CNN
+F 1 "PWR_FLAG" H 900 1550 50  0000 C CNN
+F 2 "" H 900 1400 50  0001 C CNN
+F 3 "" H 900 1400 50  0001 C CNN
+	1    900  1400
+	-1   0    0    1
+$EndComp
 $EndSCHEMATC

Commit message: replaced OPA4172IPW with OPA4172IDR
Fixes #6
Parts:
- U702, U703: MFP OPA4172IPW -> OPA4172IDR
Changed lines of the file:
@@
 F 1 "OPA4172" H 4800 1300 50  0000 L CNN
 F 2 "Housings_SOIC:SOIC-14_3.9x8.7mm_Pitch1.27mm" H 4750 1600 50  0001 C CNN
-F 3 "https://octopart.com/click/track?ct=datasheets&hlid=24903050&ppid=47153708&sid=370&sig=0f23e7a" H 4850 1700 50  0001 C CNN
+F 3 "https://octopart.com/click/track?ct=datasheets&hlid=24903049&ppid=47153707&sid=370&sig=086dfac" H 4850 1700 50  0001 C CNN
 F 4 "Texas Instruments" H 4800 1500 60  0001 C CNN "MFN"
-F 5 "OPA4172IPW" H 4800 1500 60  0001 C CNN "MFP"
+F 5 "OPA4172IDR" H 4800 1500 60  0001 C CNN "MFP"
 	2    4800 1500
 	1    0    0    -1
@@
 F 1 "OPA4172" H 9200 1300 50  0000 L CNN
 F 2 "Housings_SOIC:SOIC-14_3.9x8.7mm_Pitch1.27mm" H 9150 1600 50  0001 C CNN
-F 3 "https://octopart.com/click/track?ct=datasheets&hlid=24903050&ppid=47153708&sid=370&sig=0f23e7a" H 9250 1700 50  0001 C CNN
+F 3 "https://octopart.com/click/track?ct=datasheets&hlid=24903049&ppid=47153707&sid=370&sig=086dfac" H 9250 1700 50  0001 C CNN
 F 4 "Texas Instruments" H 9200 1800 50  0001 C CNN "MFN"
-F 5 "OPA4172IPW" H 9200 1800 50  0001 C CNN "MFP"
+F 5 "OPA4172IDR" H 9200 1800 50  0001 C CNN "MFP"
 	4    9200 1500
 	1    0    0    -1
@@
 F 1 "OPA4172" H 4800 3000 50  0000 L CNN
 F 2 "Housings_SOIC:SOIC-14_3.9x8.7mm_Pitch1.27mm" H 4750 3300 50  0001 C CNN
-F 3 "https://octopart.com/click/track?ct=datasheets&hlid=24903050&ppid=47153708&sid=370&sig=0f23e7a" H 4850 3400 50  0001 C CNN
+F 3 "https://octopart.com/click/track?ct=datasheets&hlid=24903049&ppid=47153707&sid=370&sig=086dfac" H 4850 3400 50  0001 C CNN
 F 4 "Texas Instruments" H 4800 3500 50  0001 C CNN "MFN"
-F 5 "OPA4172IPW" H 4800 3500 50  0001 C CNN "MFP"
+F 5 "OPA4172IDR" H 4800 3500 50  0001 C CNN "MFP"
 	2    4800 3200
 	1    0    0    -1
@@
 F 1 "OPA4172" H 2600 1300 50  0000 L CNN
 F 2 "Housings_SOIC:SOIC-14_3.9x8.7mm_Pitch1.27mm" H 2550 1600 50  0001 C CNN
-F 3 "https://octopart.com/click/track?ct=datasheets&hlid=24903050&ppid=47153708&sid=370&sig=0f23e7a" H 2650 1700 50  0001 C CNN
+F 3 "https://octopart.com/click/track?ct=datasheets&hlid=24903049&ppid=47153707&sid=370&sig=086dfac" H 2650 1700 50  0001 C CNN
 F 4 "Texas Instruments" H 2600 1800 50  0001 C CNN "MFN"
-F 5 "OPA4172IPW" H 2600 1800 50  0001 C CNN "MFP"
+F 5 "OPA4172IDR" H 2600 1800 50  0001 C CNN "MFP"
 	1    2600 1500
 	1    0    0    -1
@@
 F 1 "OPA4172" H 7000 1300 50  0000 L CNN
 F 2 "Housings_SOIC:SOIC-14_3.9x8.7mm_Pitch1.27mm" H 6950 1600 50  0001 C CNN
-F 3 "https://octopart.com/click/track?ct=datasheets&hlid=24903050&ppid=47153708&sid=370&sig=0f23e7a" H 7050 1700 50  0001 C CNN
+F 3 "https://octopart.com/click/track?ct=datasheets&hlid=24903049&ppid=47153707&sid=370&sig=086dfac" H 7050 1700 50  0001 C CNN
 F 4 "Texas Instruments" H 7000 1800 50  0001 C CNN "MFN"
-F 5 "OPA4172IPW" H 7000 1800 50  0001 C CNN "MFP"
+F 5 "OPA4172IDR" H 7000 1800 50  0001 C CNN "MFP"
 	3    7000 1500
 	1    0    0    -1
@@
 F 1 "OPA4172" H 2600 3000 50  0000 L CNN
 F 2 "Housings_SOIC:SOIC-14_3.9x8.7mm_Pitch1.27mm" H 2550 3300 50  0001 C CNN
-F 3 "https://octopart.com/click/track?ct=datasheets&hlid=24903050&ppid=47153708&sid=370&sig=0f23e7a" H 2650 3400 50  0001 C CNN
+F 3 "https://octopart.com/click/track?ct=datasheets&hlid=24903049&ppid=47153707&sid=370&sig=086dfac" H 2650 3400 50  0001 C CNN
 F 4 "Texas Instruments" H 2600 3500 50  0001 C CNN "MFN"
-F 5 "OPA4172IPW" H 2600 3500 50  0001 C CNN "MFP"
+F 5 "OPA4172IDR" H 2600 3500 50  0001 C CNN "MFP"
 	1    2600 3200
 	1    0    0    -1
@@
 F 1 "OPA4172" H 7000 3000 50  0000 L CNN
 F 2 "Housings_SOIC:SOIC-14_3.9x8.7mm_Pitch1.27mm" H 6950 3300 50  0001 C CNN
-F 3 "https://octopart.com/click/track?ct=datasheets&hlid=24903050&ppid=47153708&sid=370&sig=0f23e7a" H 7050 3400 50  0001 C CNN
+F 3 "https://octopart.com/click/track?ct=datasheets&hlid=24903049&ppid=47153707&sid=370&sig=086dfac" H 7050 3400 50  0001 C CNN
 F 4 "Texas Instruments" H 7000 3500 50  0001 C CNN "MFN"
-F 5 "OPA4172IPW" H 7000 3500 50  0001 C CNN "MFP"
+F 5 "OPA4172IDR" H 7000 3500 50  0001 C CNN "MFP"
 	3    7000 3200
 	1    0    0    -1
@@
 F 1 "OPA4172" H 9200 3000 50  0000 L CNN
 F 2 "Housings_SOIC:SOIC-14_3.9x8.7mm_Pitch1.27mm" H 9150 3300 50  0001 C CNN
-F 3 "https://octopart.com/click/track?ct=datasheets&hlid=24903050&ppid=47153708&sid=370&sig=0f23e7a" H 9250 3400 50  0001 C CNN
+F 3 "https://octopart.com/click/track?ct=datasheets&hlid=24903049&ppid=47153707&sid=370&sig=086dfac" H 9250 3400 50  0001 C CNN
 F 4 "Texas Instruments" H 9200 3500 50  0001 C CNN "MFN"
-F 5 "OPA4172IPW" H 9200 3500 50  0001 C CNN "MFP"
+F 5 "OPA4172IDR" H 9200 3500 50  0001 C CNN "MFP"
 	4    9200 3200
 	1    0    0    -1
