File: dac.sch (KiCad schematic (older format))
At the start: 46 parts, among them U701 DAC8568C, U702 OPA4172, U703 OPA4172

Commit message: work in progress
Parts:
- C701, C702, C703, C704, C705, C706, C707, C708, C709, C710, C711, C712, C714, C715, C717: footprint Capacitors_SMD:C_0603 -> Capacitors_SMD:C_0603_HandSoldering
- R701, R702, R703, R704, R705, R706, R707, R708, R709, R710, R711, R712, R713, R714, R715, R716, R717, R718, R719, R720, R721, R722, R723, R724, R725, R726: footprint Resistors_SMD:R_0603 -> Resistors_SMD:R_0603_HandSoldering

Commit message: work in progress
Parts:
- C701, C702, C703, C704, C705, C706, C707, C708, C709, C710, C711, C712, C714, C715, C717: footprint Capacitors_SMD:C_0603_HandSoldering -> w_capacitor:C_0603
- C713, C716: footprint Capacitors_SMD:C_0805 -> w_capacitor:C_0805
- R701, R702, R703, R704, R705, R706, R707, R708, R709, R710, R711, R712, R713, R714, R715, R716, R717, R718, R719, R720, R721, R722, R723, R724, R725, R726: footprint Resistors_SMD:R_0603_HandSoldering -> w_resistor:R_0603
