File: button-matrix.sch (KiCad schematic (older format))
At the start: 85 parts, among them SW301 TL1105T, SW302 TL1105T, SW303 TL1105T, SW304 TL1105T, SW305 TL1105T, SW306 TL1105T, SW307 TL1105T, SW308 TL1105T, SW309 TL1105T, SW310 TL1105T, SW311 TL1105T, SW312 TL1105T, SW313 TL1105T, SW314 TL1105T, SW315 TL1105T, SW316 TL1105T, SW317 TL1105T, SW318 TL1105T, SW319 TL1105T, SW320 TL1105T, SW321 TL1105T, SW322 TL1105T, SW323 TL1105T, SW324 TL1105T, SW325 TL1105T, SW326 TL1105T, SW327 TL1105T, SW328 TL1105T, SW329 TL1105T, SW330 TL1105T, SW331 TL1105T, SW332 TL1105T, SW333 TL1105T, SW334 TL1105T, SW335 TL1105T, SW336 TL1105T, SW337 TL1105T, SW338 TL1105T, SW339 TL1105T, SW340 TL1105T

Commit message: work in progress
Parts:
- removed D306, D307, D308: 1N4148, Diodes_SMD:D_SOD-123, symbol D
- removed SW306, SW307, SW308: TL1105T, w_switch:TL1105T, symbol TL1105T
- R301, R302, R303, R304, R305: MFN (none) -> Panasonic; MFP (none) -> ERJ-3EKF1002V
Changed lines of the file:
@@
-$EndComp
-$Comp
-L TL1105T SW306
-U 1 1 59D960E9
-P 6450 1900
-F 0 "SW306" H 6450 1700 50  0000 C CNN
-F 1 "TL1105T" H 6450 2100 50  0000 C CNN
-F 2 "w_switch:TL1105T" H 6350 1900 50  0001 C CNN
-F 3 "http://datasheet.octopart.com/TL1105TF160Q-E-Switch-datasheet-502092.pdf" H 6350 1900 50  0001 C CNN
-F 4 "E-Switch" H 6450 1800 50  0001 C CNN "MFN"
-F 5 "TL1105TF160Q" H 6450 1800 50  0001 C CNN "MFP"
-	1    6450 1900
-	1    0    0    -1
-$EndComp
-$Comp
-L D D306
-U 1 1 59D9610F
-P 6800 1650
-F 0 "D306" H 6800 1750 50  0000 C CNN
-F 1 "1N4148" H 6800 1550 50  0000 C CNN
-F 2 "Diodes_SMD:D_SOD-123" H 6800 1650 50  0001 C CNN
-F 3 "http://datasheet.octopart.com/1N4148W-7-F-Diodes-Inc.-datasheet-12518151.pdf" H 6800 1650 50  0001 C CNN
-F 4 "Diodes Inc." H 6800 1850 50  0001 C CNN "MFN"
-F 5 "1N4148W-7-F" H 6800 1850 50  0001 C CNN "MFP"
-	1    6800 1650
-	0    -1   -1   0
 $EndComp
 $Comp
@@
 $EndComp
 $Comp
-L TL1105T SW307
-U 1 1 59D96151
-P 7250 1900
-F 0 "SW307" H 7250 1700 50  0000 C CNN
-F 1 "TL1105T" H 7250 2100 50  0000 C CNN
-F 2 "w_switch:TL1105T" H 7150 1900 50  0001 C CNN
-F 3 "http://datasheet.octopart.com/TL1105TF160Q-E-Switch-datasheet-502092.pdf" H 7150 1900 50  0001 C CNN
-F 4 "E-Switch" H 7250 1800 50  0001 C CNN "MFN"
-F 5 "TL1105TF160Q" H 7250 1800 50  0001 C CNN "MFP"
-	1    7250 1900
-	1    0    0    -1
-$EndComp
-$Comp
-L D D307
-U 1 1 59D96177
-P 7600 1650
-F 0 "D307" H 7600 1750 50  0000 C CNN
-F 1 "1N4148" H 7600 1550 50  0000 C CNN
-F 2 "Diodes_SMD:D_SOD-123" H 7600 1650 50  0001 C CNN
-F 3 "http://datasheet.octopart.com/1N4148W-7-F-Diodes-Inc.-datasheet-12518151.pdf" H 7600 1650 50  0001 C CNN
-F 4 "Diodes Inc." H 7600 1850 50  0001 C CNN "MFN"
-F 5 "1N4148W-7-F" H 7600 1850 50  0001 C CNN "MFP"
-	1    7600 1650
-	0    -1   -1   0
-$EndComp
-$Comp
 L D D315
 U 1 1 59D9617D
@@
 $EndComp
 $Comp
-L TL1105T SW308
-U 1 1 59D961B9
-P 8050 1900
-F 0 "SW308" H 8050 1700 50  0000 C CNN
-F 1 "TL1105T" H 8050 2100 50  0000 C CNN
-F 2 "w_switch:TL1105T" H 7950 1900 50  0001 C CNN
-F 3 "http://datasheet.octopart.com/TL1105TF160Q-E-Switch-datasheet-502092.pdf" H 7950 1900 50  0001 C CNN
-F 4 "E-Switch" H 8050 1800 50  0001 C CNN "MFN"
-F 5 "TL1105TF160Q" H 8050 1800 50  0001 C CNN "MFP"
-	1    8050 1900
-	1    0    0    -1
-$EndComp
-$Comp
-L D D308
-U 1 1 59D961DF
-P 8400 1650
-F 0 "D308" H 8400 1750 50  0000 C CNN
-F 1 "1N4148" H 8400 1550 50  0000 C CNN
-F 2 "Diodes_SMD:D_SOD-123" H 8400 1650 50  0001 C CNN
-F 3 "http://datasheet.octopart.com/1N4148W-7-F-Diodes-Inc.-datasheet-12518151.pdf" H 8400 1650 50  0001 C CNN
-F 4 "Diodes Inc." H 8400 1850 50  0001 C CNN "MFN"
-F 5 "1N4148W-7-F" H 8400 1850 50  0001 C CNN "MFP"
-	1    8400 1650
-	0    -1   -1   0
-$EndComp
-$Comp
 L D D316
 U 1 1 59D961E5
@@
 F 1 "10k" V 8700 1750 50  0000 C CNN
 F 2 "Resistors_SMD:R_0603" V 8630 1750 50  0001 C CNN
-F 3 "" H 8700 1750 50  0001 C CNN
+F 3 "http://datasheet.octopart.com/ERJ-3EKF1002V-Panasonic-datasheet-13266541.pdf" H 8700 1750 50  0001 C CNN
+F 4 "Panasonic" H 8780 1850 50  0001 C CNN "MFN"
+F 5 "ERJ-3EKF1002V" H 8780 1850 50  0001 C CNN "MFP"
 	1    8700 1750
 	1    0    0    -1
@@
 F 1 "10k" V 8700 2450 50  0000 C CNN
 F 2 "Resistors_SMD:R_0603" V 8630 2450 50  0001 C CNN
-F 3 "" H 8700 2450 50  0001 C CNN
+F 3 "http://datasheet.octopart.com/ERJ-3EKF1002V-Panasonic-datasheet-13266541.pdf" H 8700 2450 50  0001 C CNN
+F 4 "Panasonic" H 8780 2550 50  0001 C CNN "MFN"
+F 5 "ERJ-3EKF1002V" H 8780 2550 50  0001 C CNN "MFP"
 	1    8700 2450
 	1    0    0    -1
@@
 F 1 "10k" V 8700 3150 50  0000 C CNN
 F 2 "Resistors_SMD:R_0603" V 8630 3150 50  0001 C CNN
-F 3 "" H 8700 3150 50  0001 C CNN
+F 3 "http://datasheet.octopart.com/ERJ-3EKF1002V-Panasonic-datasheet-13266541.pdf" H 8700 3150 50  0001 C CNN
+F 4 "Panasonic" H 8780 3250 50  0001 C CNN "MFN"
+F 5 "ERJ-3EKF1002V" H 8780 3250 50  0001 C CNN "MFP"
 	1    8700 3150
 	1    0    0    -1
@@
 F 1 "10k" V 8700 3850 50  0000 C CNN
 F 2 "Resistors_SMD:R_0603" V 8630 3850 50  0001 C CNN
-F 3 "" H 8700 3850 50  0001 C CNN
+F 3 "http://datasheet.octopart.com/ERJ-3EKF1002V-Panasonic-datasheet-13266541.pdf" H 8700 3850 50  0001 C CNN
+F 4 "Panasonic" H 8780 3950 50  0001 C CNN "MFN"
+F 5 "ERJ-3EKF1002V" H 8780 3950 50  0001 C CNN "MFP"
 	1    8700 3850
 	1    0    0    -1
@@
 F 1 "10k" V 8700 4550 50  0000 C CNN
 F 2 "Resistors_SMD:R_0603" V 8630 4550 50  0001 C CNN
-F 3 "" H 8700 4550 50  0001 C CNN
+F 3 "http://datasheet.octopart.com/ERJ-3EKF1002V-Panasonic-datasheet-13266541.pdf" H 8700 4550 50  0001 C CNN
+F 4 "Panasonic" H 8780 4650 50  0001 C CNN "MFN"
+F 5 "ERJ-3EKF1002V" H 8780 4650 50  0001 C CNN "MFP"
 	1    8700 4550
 	1    0    0    -1
@@
 	6000 4800 5900 4800
 Wire Wire Line
-	6100 1800 6100 5200
-Wire Wire Line
-	6200 1800 6100 1800
-Wire Wire Line
-	6200 2000 6100 2000
-Wire Wire Line
 	6200 2500 6100 2500
 Wire Wire Line
@@
 	6200 4800 6100 4800
 Wire Wire Line
-	6700 1800 6800 1800
-Wire Wire Line
-	6800 1800 6800 2000
-Wire Wire Line
-	6800 2000 6700 2000
-Wire Wire Line
 	6700 2500 6800 2500
 Wire Wire Line
@@
 	6800 4800 6700 4800
 Wire Wire Line
-	6900 1800 6900 5200
-Wire Wire Line
-	7000 1800 6900 1800
-Wire Wire Line
-	7000 2000 6900 2000
-Wire Wire Line
 	7000 2500 6900 2500
 Wire Wire Line
@@
 	7000 4800 6900 4800
 Wire Wire Line
-	7500 1800 7600 1800
-Wire Wire Line
-	7600 1800 7600 2000
-Wire Wire Line
-	7600 2000 7500 2000
-Wire Wire Line
 	7500 2500 7600 2500
 Wire Wire Line
@@
 	7600 4800 7500 4800
 Wire Wire Line
-	7700 1800 7700 5200
-Wire Wire Line
-	7800 1800 7700 1800
-Wire Wire Line
-	7800 2000 7700 2000
-Wire Wire Line
 	7800 2500 7700 2500
 Wire Wire Line
@@
 Wire Wire Line
 	7800 4800 7700 4800
-Wire Wire Line
-	8300 1800 8400 1800
-Wire Wire Line
-	8400 1800 8400 2000
-Wire Wire Line
-	8400 2000 8300 2000
 Wire Wire Line
 	8300 2500 8400 2500
@@
 Connection ~ 5300 4600
 Connection ~ 5300 4800
-Connection ~ 6100 2000
 Connection ~ 6100 2500
 Connection ~ 6100 2700
@@
 Connection ~ 6100 4600
 Connection ~ 6100 4800
-Connection ~ 6900 2000
 Connection ~ 6900 2500
 Connection ~ 6900 2700
@@
 Connection ~ 6900 4600
 Connection ~ 6900 4800
-Connection ~ 7700 2000
 Connection ~ 7700 2500
 Connection ~ 7700 2700
@@
 Connection ~ 5200 1500
 Connection ~ 6000 1500
-Connection ~ 6800 1500
-Connection ~ 7600 1500
-Connection ~ 8400 1500
 Connection ~ 3600 2200
 Connection ~ 4400 2200
@@
 Connection ~ 8900 3400
 Connection ~ 8900 4100
+Wire Wire Line
+	6100 2500 6100 5200
+Wire Wire Line
+	6900 2500 6900 5200
+Wire Wire Line
+	7700 2500 7700 5200
 $EndSCHEMATC

Commit message: work in progress
Parts:
- removed R301, R302, R303, R304, R305: 10k, Resistors_SMD:R_0603, symbol R
Other:
- moved on the sheet: D301, D302, D303, D304, D309, D310, D311, D312, D314, D315, D316, D317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

Commit message: cleanup
Parts:
- D301, D302, D303, D304, D305, D309, D310, D311, D312, D313, D314, D315, D316, D317, D318, D319, D320, D321, D322, D323, D324, D325, D326, D327, D328, D329, D330, D331, D332, D333, D334, D335, D336, D337, D338, D339, D340: footprint Diodes_SMD:D_SOD-123 -> w_diode:D_SOD-123
