File: button-matrix.sch (KiCad schematic (older format))
At the start: 74 parts, among them SW1 TL1105, SW10 TL1105, SW11 TL1105, SW12 TL1105, SW13 TL1105, SW14 TL1105, SW15 TL1105, SW16 TL1105, SW17 TL1105, SW18 TL1105, SW2 TL1105, SW20 TL1105, SW21 TL1105, SW22 TL1105, SW23 TL1105, SW24 TL1105, SW25 TL1105, SW26 TL1105, SW27 TL1105, SW28 TL1105, SW29 TL1105, SW3 TL1105, SW30 TL1105, SW31 TL1105, SW32 TL1105, SW33 TL1105, SW34 TL1105, SW35 TL1105, SW36 TL1105, SW37 TL1105, SW38 TL1105, SW39 TL1105, SW4 TL1105, SW5 TL1105, SW6 TL1105, SW7 TL1105, SW9 TL1105

Commit message: added package field
Parts:
- D10, D11, D12, D13, D14, D15, D16, D17, D18, D19, D20, D21, D22, D23, D24, D25, D26, D27, D28, D29, D30, D31, D32, D33, D34, D35, D36, D37, D38, D39, D40, D41, D5, D6, D7, D8, D9: Package (none) -> SOD-123
Changed lines of the file:
@@
 F 4 "Diodes Inc." H 2400 1850 50  0001 C CNN "MFN"
 F 5 "1N4148W-7-F" H 2400 1850 50  0001 C CNN "MFP"
+F 6 "SOD-123" H 2400 1850 50  0001 C CNN "Package"
 	1    2400 1650
 	0    -1   -1   0
@@
 F 4 "Diodes Inc." H 2400 2550 50  0001 C CNN "MFN"
 F 5 "1N4148W-7-F" H 2400 2550 50  0001 C CNN "MFP"
+F 6 "SOD-123" H 2400 2550 50  0001 C CNN "Package"
 	1    2400 2350
 	0    -1   -1   0
@@
 F 4 "Diodes Inc." H 2400 3250 50  0001 C CNN "MFN"
 F 5 "1N4148W-7-F" H 2400 3250 50  0001 C CNN "MFP"
+F 6 "SOD-123" H 2400 3250 50  0001 C CNN "Package"
 	1    2400 3050
 	0    -1   -1   0
@@
 F 4 "Diodes Inc." H 2400 3950 50  0001 C CNN "MFN"
 F 5 "1N4148W-7-F" H 2400 3950 50  0001 C CNN "MFP"
+F 6 "SOD-123" H 2400 3950 50  0001 C CNN "Package"
 	1    2400 3750
 	0    -1   -1   0
@@
 F 4 "Diodes Inc." H 2400 4650 50  0001 C CNN "MFN"
 F 5 "1N4148W-7-F" H 2400 4650 50  0001 C CNN "MFP"
+F 6 "SOD-123" H 2400 4650 50  0001 C CNN "Package"
 	1    2400 4450
 	0    -1   -1   0
@@
 F 4 "Diodes Inc." H 3300 1850 50  0001 C CNN "MFN"
 F 5 "1N4148W-7-F" H 3300 1850 50  0001 C CNN "MFP"
+F 6 "SOD-123" H 3300 1850 50  0001 C CNN "Package"
 	1    3300 1650
 	0    -1   -1   0
@@
 F 4 "Diodes Inc." H 3300 2550 50  0001 C CNN "MFN"
 F 5 "1N4148W-7-F" H 3300 2550 50  0001 C CNN "MFP"
+F 6 "SOD-123" H 3300 2550 50  0001 C CNN "Package"
 	1    3300 2350
 	0    -1   -1   0
@@
 F 4 "Diodes Inc." H 3300 3250 50  0001 C CNN "MFN"
 F 5 "1N4148W-7-F" H 3300 3250 50  0001 C CNN "MFP"
+F 6 "SOD-123" H 3300 3250 50  0001 C CNN "Package"
 	1    3300 3050
 	0    -1   -1   0
@@
 F 4 "Diodes Inc." H 3300 3950 50  0001 C CNN "MFN"
 F 5 "1N4148W-7-F" H 3300 3950 50  0001 C CNN "MFP"
+F 6 "SOD-123" H 3300 3950 50  0001 C CNN "Package"
 	1    3300 3750
 	0    -1   -1   0
@@
 F 4 "Diodes Inc." H 3300 4650 50  0001 C CNN "MFN"
 F 5 "1N4148W-7-F" H 3300 4650 50  0001 C CNN "MFP"
+F 6 "SOD-123" H 3300 4650 50  0001 C CNN "Package"
 	1    3300 4450
 	0    -1   -1   0
@@
 F 4 "Diodes Inc." H 4200 1850 50  0001 C CNN "MFN"
 F 5 "1N4148W-7-F" H 4200 1850 50  0001 C CNN "MFP"
+F 6 "SOD-123" H 4200 1850 50  0001 C CNN "Package"
 	1    4200 1650
 	0    -1   -1   0
@@
 F 4 "Diodes Inc." H 4200 2550 50  0001 C CNN "MFN"
 F 5 "1N4148W-7-F" H 4200 2550 50  0001 C CNN "MFP"
+F 6 "SOD-123" H 4200 2550 50  0001 C CNN "Package"
 	1    4200 2350
 	0    -1   -1   0
@@
 F 4 "Diodes Inc." H 4200 3250 50  0001 C CNN "MFN"
 F 5 "1N4148W-7-F" H 4200 3250 50  0001 C CNN "MFP"
+F 6 "SOD-123" H 4200 3250 50  0001 C CNN "Package"
 	1    4200 3050
 	0    -1   -1   0
@@
 F 4 "Diodes Inc." H 4200 3950 50  0001 C CNN "MFN"
 F 5 "1N4148W-7-F" H 4200 3950 50  0001 C CNN "MFP"
+F 6 "SOD-123" H 4200 3950 50  0001 C CNN "Package"
 	1    4200 3750
 	0    -1   -1   0
@@
 F 4 "Diodes Inc." H 4200 4650 50  0001 C CNN "MFN"
 F 5 "1N4148W-7-F" H 4200 4650 50  0001 C CNN "MFP"
+F 6 "SOD-123" H 4200 4650 50  0001 C CNN "Package"
 	1    4200 4450
 	0    -1   -1   0
@@
 F 4 "Diodes Inc." H 5100 1850 50  0001 C CNN "MFN"
 F 5 "1N4148W-7-F" H 5100 1850 50  0001 C CNN "MFP"
+F 6 "SOD-123" H 5100 1850 50  0001 C CNN "Package"
 	1    5100 1650
 	0    -1   -1   0
@@
 F 4 "Diodes Inc." H 5100 2550 50  0001 C CNN "MFN"
 F 5 "1N4148W-7-F" H 5100 2550 50  0001 C CNN "MFP"
+F 6 "SOD-123" H 5100 2550 50  0001 C CNN "Package"
 	1    5100 2350
 	0    -1   -1   0
@@
 F 4 "Diodes Inc." H 5100 3250 50  0001 C CNN "MFN"
 F 5 "1N4148W-7-F" H 5100 3250 50  0001 C CNN "MFP"
+F 6 "SOD-123" H 5100 3250 50  0001 C CNN "Package"
 	1    5100 3050
 	0    -1   -1   0
@@
 F 4 "Diodes Inc." H 5100 3950 50  0001 C CNN "MFN"
 F 5 "1N4148W-7-F" H 5100 3950 50  0001 C CNN "MFP"
+F 6 "SOD-123" H 5100 3950 50  0001 C CNN "Package"
 	1    5100 3750
 	0    -1   -1   0
@@
 F 4 "Diodes Inc." H 5100 4650 50  0001 C CNN "MFN"
 F 5 "1N4148W-7-F" H 5100 4650 50  0001 C CNN "MFP"
+F 6 "SOD-123" H 5100 4650 50  0001 C CNN "Package"
 	1    5100 4450
 	0    -1   -1   0
@@
 F 4 "Diodes Inc." H 6000 1850 50  0001 C CNN "MFN"
 F 5 "1N4148W-7-F" H 6000 1850 50  0001 C CNN "MFP"
+F 6 "SOD-123" H 6000 1850 50  0001 C CNN "Package"
 	1    6000 1650
 	0    -1   -1   0
@@
 F 4 "Diodes Inc." H 6000 2550 50  0001 C CNN "MFN"
 F 5 "1N4148W-7-F" H 6000 2550 50  0001 C CNN "MFP"
+F 6 "SOD-123" H 6000 2550 50  0001 C CNN "Package"
 	1    6000 2350
 	0    -1   -1   0
@@
 F 4 "Diodes Inc." H 6000 3250 50  0001 C CNN "MFN"
 F 5 "1N4148W-7-F" H 6000 3250 50  0001 C CNN "MFP"
+F 6 "SOD-123" H 6000 3250 50  0001 C CNN "Package"
 	1    6000 3050
 	0    -1   -1   0
@@
 F 4 "Diodes Inc." H 6000 3950 50  0001 C CNN "MFN"
 F 5 "1N4148W-7-F" H 6000 3950 50  0001 C CNN "MFP"
+F 6 "SOD-123" H 6000 3950 50  0001 C CNN "Package"
 	1    6000 3750
 	0    -1   -1   0
@@
 F 4 "Diodes Inc." H 6000 4650 50  0001 C CNN "MFN"
 F 5 "1N4148W-7-F" H 6000 4650 50  0001 C CNN "MFP"
+F 6 "SOD-123" H 6000 4650 50  0001 C CNN "Package"
 	1    6000 4450
 	0    -1   -1   0
@@
 F 4 "Diodes Inc." H 6900 2550 50  0001 C CNN "MFN"
 F 5 "1N4148W-7-F" H 6900 2550 50  0001 C CNN "MFP"
+F 6 "SOD-123" H 6900 2550 50  0001 C CNN "Package"
 	1    6900 2350
 	0    -1   -1   0
@@
 F 4 "Diodes Inc." H 6900 3250 50  0001 C CNN "MFN"
 F 5 "1N4148W-7-F" H 6900 3250 50  0001 C CNN "MFP"
+F 6 "SOD-123" H 6900 3250 50  0001 C CNN "Package"
 	1    6900 3050
 	0    -1   -1   0
@@
 F 4 "Diodes Inc." H 6900 3950 50  0001 C CNN "MFN"
 F 5 "1N4148W-7-F" H 6900 3950 50  0001 C CNN "MFP"
+F 6 "SOD-123" H 6900 3950 50  0001 C CNN "Package"
 	1    6900 3750
 	0    -1   -1   0
@@
 F 4 "Diodes Inc." H 6900 4650 50  0001 C CNN "MFN"
 F 5 "1N4148W-7-F" H 6900 4650 50  0001 C CNN "MFP"
+F 6 "SOD-123" H 6900 4650 50  0001 C CNN "Package"
 	1    6900 4450
 	0    -1   -1   0
@@
 F 4 "Diodes Inc." H 7800 2550 50  0001 C CNN "MFN"
 F 5 "1N4148W-7-F" H 7800 2550 50  0001 C CNN "MFP"
+F 6 "SOD-123" H 7800 2550 50  0001 C CNN "Package"
 	1    7800 2350
 	0    -1   -1   0
@@
 F 4 "Diodes Inc." H 7800 3250 50  0001 C CNN "MFN"
 F 5 "1N4148W-7-F" H 7800 3250 50  0001 C CNN "MFP"
+F 6 "SOD-123" H 7800 3250 50  0001 C CNN "Package"
 	1    7800 3050
 	0    -1   -1   0
@@
 F 4 "Diodes Inc." H 7800 3950 50  0001 C CNN "MFN"
 F 5 "1N4148W-7-F" H 7800 3950 50  0001 C CNN "MFP"
+F 6 "SOD-123" H 7800 3950 50  0001 C CNN "Package"
 	1    7800 3750
 	0    -1   -1   0
@@
 F 4 "Diodes Inc." H 7800 4650 50  0001 C CNN "MFN"
 F 5 "1N4148W-7-F" H 7800 4650 50  0001 C CNN "MFP"
+F 6 "SOD-123" H 7800 4650 50  0001 C CNN "Package"
 	1    7800 4450
 	0    -1   -1   0
@@
 F 4 "Diodes Inc." H 8700 2550 50  0001 C CNN "MFN"
 F 5 "1N4148W-7-F" H 8700 2550 50  0001 C CNN "MFP"
+F 6 "SOD-123" H 8700 2550 50  0001 C CNN "Package"
 	1    8700 2350
 	0    -1   -1   0
@@
 F 4 "Diodes Inc." H 8700 3250 50  0001 C CNN "MFN"
 F 5 "1N4148W-7-F" H 8700 3250 50  0001 C CNN "MFP"
+F 6 "SOD-123" H 8700 3250 50  0001 C CNN "Package"
 	1    8700 3050
 	0    -1   -1   0
@@
 F 4 "Diodes Inc." H 8700 3950 50  0001 C CNN "MFN"
 F 5 "1N4148W-7-F" H 8700 3950 50  0001 C CNN "MFP"
+F 6 "SOD-123" H 8700 3950 50  0001 C CNN "Package"
 	1    8700 3750
 	0    -1   -1   0
@@
 F 4 "Diodes Inc." H 8700 4650 50  0001 C CNN "MFN"
 F 5 "1N4148W-7-F" H 8700 4650 50  0001 C CNN "MFP"
+F 6 "SOD-123" H 8700 4650 50  0001 C CNN "Package"
 	1    8700 4450
 	0    -1   -1   0

Commit message: cleaned up schematics
Other:
- note added: "BUTTON MATRIX"
Changed lines of the file:
@@
 Sheet 4 8
 Title "per|former eurorack sequencer"
-Date "2018-08-26"
-Rev "0.3"
+Date "2018-10-09"
+Rev "1.0"
 Comp "westlicht"
 Comment1 "cc-by-sa"
@@
 Connection ~ 7800 4300
 Connection ~ 8700 4300
+Wire Notes Line
+	600  600  600  6400
+Wire Notes Line
+	600  6400 11100 6400
+Wire Notes Line
+	11100 6400 11100 600
+Wire Notes Line
+	11100 600  600  600
+Text Notes 700  6300 0    51   ~ 0
+BUTTON MATRIX
 $EndSCHEMATC

Commit message: updated schematics to kicad5
Parts:
- D10, D11, D12, D13, D14, D15, D16, D17, D18, D19, D20, D21, D22, D23, D24, D25, D26, D27, D28, D29, D30, D31, D32, D33, D34, D35, D36, D37, D38, D39, D40, D41, D5, D6, D7, D8, D9: symbol D -> Device:D
- SW1, SW10, SW11, SW12, SW13, SW14, SW15, SW16, SW17, SW18, SW2, SW20, SW21, SW22, SW23, SW24, SW25, SW26, SW27, SW28, SW29, SW3, SW30, SW31, SW32, SW33, SW34, SW35, SW36, SW37, SW38, SW39, SW4, SW5, SW6, SW7, SW9: symbol TL1105T -> w_switch:TL1105T
