File: frontpanel.kicad_pcb (KiCad board)
At the start: 2 copper layers, 172.7 x 128.3 mm, 107 parts, among them J102 NHD-3.12-25664UC, SW309 TL1105T, SW310 TL1105T, SW311 TL1105T, SW312 TL1105T, SW313 TL1105T, SW314 TL1105T, SW315 TL1105T, SW316 TL1105T, SW317 TL1105T, SW318 TL1105T, SW319 TL1105T, SW320 TL1105T, SW321 TL1105T, SW322 TL1105T, SW323 TL1105T, SW324 TL1105T, SW325 TL1105T, SW326 TL1105T, SW327 TL1105T, SW328 TL1105T, SW329 TL1105T, SW330 TL1105T, SW331 TL1105T, SW332 TL1105T, SW333 TL1105T, SW334 TL1105T, SW335 TL1105T, SW336 TL1105T, SW337 TL1105T, SW338 TL1105T, SW339 TL1105T, SW340 TL1105T

Commit message: work on frontpanel
Parts:
- renumbered SW325 to 1, SW334 to 10, SW335 to 11, SW336 to 12, SW337 to 13, SW338 to 14, SW339 to 15, SW340 to 16, SW326 to 2, SW327 to 3, SW328 to 4, SW329 to 5, SW330 to 6, SW331 to 7, SW332 to 8, SW333 to 9, SW310 to BPM, SW313 to FILL, SW315 to MUTE, SW309 to PLAY, SW316 to SHIFT, SW314 to SNAP, SW317 to T1, SW318 to T2, SW319 to T3, SW320 to T4, SW321 to T5, SW322 to T6, SW323 to T7, SW324 to T8, SW312 to XXX, SW311 to XXX
Other:
- board size 172.7 x 128.3 mm -> 172.5 x 128.3 mm
- board text added: ".p.e.r.4.m.e.r."

Commit message: last cleanup before sending to fab
Other:
- board text added: "per|former"
- board text added: "westlicht"
- board text removed: ".p.e.r.4.m.e.r."
Changed lines of the file:
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@@
     (links 0)
     (no_connects 0)
-    (area 62.508314 24.5476 255.368115 158.2524)
+    (area 76.124999 27.229999 248.775001 155.650001)
     (thickness 1.6)
-    (drawings 21)
+    (drawings 30)
     (tracks 0)
     (zones 0)
@@
     (45 Margin user)
     (46 B.CrtYd user)
-    (47 F.CrtYd user)
+    (47 F.CrtYd user hide)
     (48 B.Fab user)
     (49 F.Fab user hide)
@@
     (visible_elements FFFFFF7F)
     (pcbplotparams
-      (layerselection 0x00030_80000001)
+      (layerselection 0x01020_00000000)
       (usegerberextensions false)
       (excludeedgelayer true)
@@
       (outputformat 1)
       (mirror false)
-      (drillshape 1)
+      (drillshape 0)
       (scaleselection 1)
       (outputdirectory ""))
@@
     (at 86.36 76.2)
     (tags "rotary, encoder, ALPS")
-    (fp_text reference DATA (at 0 -10.16) (layer F.SilkS)
+    (fp_text reference DATA (at 0 -10.16) (layer F.SilkS) hide
       (effects (font (size 1.5 1.5) (thickness 0.25)))
     )
@@
   (module w_frontpanel:TL1105_1R_FP (layer F.Cu)
     (at 209.55 114.3)
-    (fp_text reference XXX (at 6.35 0) (layer F.SilkS)
+    (fp_text reference XXX (at 6.35 0) (layer F.SilkS) hide
       (effects (font (size 1.5 1.5) (thickness 0.25)))
     )
@@
   (module w_frontpanel:TL1105_1R_FP (layer F.Cu)
     (at 196.85 114.3)
-    (fp_text reference XXX (at 6.35 0) (layer F.SilkS)
+    (fp_text reference XXX (at 6.35 0) (layer F.SilkS) hide
       (effects (font (size 1.5 1.5) (thickness 0.25)))
     )
@@
     (pad 1 np_thru_hole circle (at 0 0) (size 2.2 2.2) (drill 2.2) (layers *.Cu *.Mask))
   )
-  (gr_text .p.e.r.4.m.e.r. (at 161.925 31.75) (layer F.SilkS)
-    (effects (font (size 4 4) (thickness 0.5)))
+  (gr_line (start 76.2 147.955) (end 248.92 147.955) (layer F.SilkS) (width 0.2))
+  (gr_line (start 76.2 34.925) (end 248.92 34.925) (layer F.SilkS) (width 0.2))
+  (gr_line (start 168.91 87.63) (end 168.91 93.98) (layer F.SilkS) (width 0.25))
+  (gr_line (start 153.67 87.63) (end 153.67 93.98) (layer F.SilkS) (width 0.25))
+  (gr_line (start 138.43 87.63) (end 138.43 93.98) (layer F.SilkS) (width 0.25))
+  (gr_line (start 123.19 87.63) (end 123.19 93.98) (layer F.SilkS) (width 0.25))
+  (gr_line (start 107.95 87.63) (end 107.95 93.98) (layer F.SilkS) (width 0.25))
+  (gr_circle (center 86.36 76.2) (end 86.36 67.945) (layer F.SilkS) (width 0.25))
+  (gr_text westlicht (at 161.925 151.765) (layer F.SilkS)
+    (effects (font (size 2 2) (thickness 0.25)))
+  )
+  (gr_text per|former (at 201.93 74.295) (layer F.SilkS)
+    (effects (font (size 4.5 4.5) (thickness 0.5)))
   )
   (gr_line (start 248.92 144.78) (end 76.2 144.78) (layer F.Fab) (width 0.2))

Commit message: work on frontpanel
Parts:
- removed the REF** at (79.4, 139.7)
- removed the REF** at (79.4, 114.3)
- removed the REF** at (187.3, 114.3)
- J601: renamed from MIDI IN
- J602: renamed from MIDI OUT
- J603: renamed from CLK IN
- J604: renamed from RST IN
- J605: renamed from CLK OUT
- J606: renamed from RST OUT
- J607: renamed from CV1 IN
- J608: renamed from CV2 IN
- J609: renamed from CV3 IN
- J610: renamed from CV4 IN
- REF**: footprint Mounting_Holes:MountingHole_2.2mm_M2 -> Mounting_Holes:MountingHole_2.2mm_M2_Pad
- moved >> 108.0 mm to (101.6, 127.0), turned to 90 degrees
- moved BPM 108.0 mm to (101.6, 101.6), turned to 90 degrees
- moved LED402 108.0 mm to (101.6, 95.2)
- moved LED404 108.0 mm to (101.6, 108.0)
- moved LED406 108.0 mm to (101.6, 120.7)
- moved LED408 108.0 mm to (101.6, 133.3)
- moved PAGE 108.0 mm to (101.6, 139.7), turned to 90 degrees
- moved PATT 108.0 mm to (101.6, 114.3), turned to 90 degrees
- moved << 107.9 mm to (88.9, 127.0), turned to 90 degrees
- moved LED401 107.9 mm to (88.9, 95.2)
- moved LED403 107.9 mm to (88.9, 108.0)
- moved LED405 107.9 mm to (88.9, 120.7)
- moved LED407 107.9 mm to (88.9, 133.3)
- moved PERF 107.9 mm to (88.9, 114.3), turned to 90 degrees
- moved PLAY 107.9 mm to (88.9, 101.6), turned to 90 degrees
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- renumbered FILL to <<, SNAP to >>, DATA to ENC101, CV1 to J611, CV2 to J612, CV3 to J613, CV4 to J614, CV5 to J615, CV6 to J616, CV7 to J617, CV8 to J618, GATE1 to J619, GATE2 to J620, GATE3 to J621, GATE4 to J622, GATE5 to J623, GATE6 to J624, GATE7 to J625, GATE8 to J626, USB to JP101, J102 to JP102, SDCARD to JP103, SHIFT to PAGE, XXX to PATT, XXX to PERF, MUTE to SHIFT, F1 to SW301, F2 to SW302, F3 to SW303, F4 to SW304, F5 to SW305, T1 to SW317, T2 to SW318, T3 to SW319, T4 to SW320, T5 to SW321, T6 to SW322, T7 to SW323, T8 to SW324, 1 to SW325, 2 to SW326, 3 to SW327, 4 to SW328, 5 to SW329, 6 to SW330, 7 to SW331, 8 to SW332, 9 to SW333, 10 to SW334, 11 to SW335, 12 to SW336, 13 to SW337, 14 to SW338, 15 to SW339, 16 to SW340
Other:
- outline, holes or cut-outs redrawn
- board text added: "+12V"
- board text added: "-12V"
- board text added: "BOOT"
- board text added: "BPM"
- board text added: "CLK IN"
- board text added: "CLK OUT"
- board text added: "CLOCK"
- board text added: "CONFIG"
- board text added: "CV1"
- board text added: "CV1 IN"
- board text added: "CV2"
- board text added: "CV2 IN"
- board text added: "CV3"
- board text added: "CV3 IN"
- board text added: "CV4"
- board text added: "CV4 IN"
- board text added: "CV5"
- board text added: "CV6"
- board text added: "CV7"
- board text added: "CV8"
- board text added: "DIVISOR"
- board text added: "EDIT"
- board text added: "F1"
- board text added: "F2"
- board text added: "F3"
- board text added: "F4"
- board text added: "F5"
- board text added: "FIRST"
- board text added: "GATE1"
- board text added: "GATE2"
- board text added: "GATE3"
- board text added: "GATE4"
- board text added: "GATE5"
- board text added: "GATE6"
- board text added: "GATE7"
- board text added: "GATE8"
- board text added: "GEN"
- board text added: "GND"
- board text added: "JTAG"
- board text added: "LAST"
- board text added: "LAYOUT"
- board text added: "LEFT"
- board text added: "MIDI IN"
- board text added: "MIDI OUT"
- board text added: "MODE"
- board text added: "MONITOR"
- board text added: "PAGE"
- board text added: "PATT"
- board text added: "PERF"
- board text added: "PLAY"
- board text added: "PROJECT"
- board text added: "RED LINE"
- board text added: "RESET"
- board text added: "RIGHT"
- board text added: "ROOT"
- board text added: "ROUTING"
- board text added: "RST IN"
- board text added: "RST OUT"
- board text added: "RX"
- board text added: "S1"
- board text added: "S10"
- board text added: "S11"
- board text added: "S12"
- board text added: "S13"
- board text added: "S14"
- board text added: "S15"
- board text added: "S16"
- board text added: "S2"
- board text added: "S3"
- board text added: "S4"
- board text added: "S5"
- board text added: "S6"
- board text added: "S7"
- board text added: "S8"
- board text added: "S9"
- board text added: "SCALE"
- board text added: "SDCARD"
- board text added: "SEQ"
- board text added: "SERIAL"
- board text added: "SHIFT"
- board text added: "SONG"
- board text added: "T1"
- board text added: "T2"
- board text added: "T3"
- board text added: "T4"
- board text added: "T5"
- board text added: "T6"
- board text added: "T7"
- board text added: "T8"
- board text added: "TRACK"
- board text added: "TX"
- board text added: "USB"
- board text added: "USERSCALE"
- board text added: "cc-by-sa Simon Kallweit 2018 board revision 0.2"

Commit message: cleanup
Parts:
- JP103: footprint w_frontpanel:PJS008U-3000-0_FP -> w_frontpanel:PJS008U-3000-0_FP_LARGER
Changed lines of the file:
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@@
     (fp_line (start -6.55 -4.225) (end 6.55 -4.225) (layer Edge.Cuts) (width 0.15))
   )
-  (module w_frontpanel:PJS008U-3000-0_FP (layer F.Cu)
+  (module w_frontpanel:PJS008U-3000-0_FP_LARGER (layer F.Cu)
     (at 86.36 53.34 180)
     (descr https://www.yamaichi.de/uploads/media/PJS008U-3000.pdf)
@@
       (effects (font (size 1 1) (thickness 0.15)))
     )
-    (fp_line (start -6.8 0.47) (end -6.8 2.77) (layer Edge.Cuts) (width 0.15))
-    (fp_line (start -6.8 2.77) (end 6 2.77) (layer Edge.Cuts) (width 0.15))
-    (fp_line (start -6.8 0.47) (end 6 0.47) (layer Edge.Cuts) (width 0.15))
-    (fp_line (start 6 0.47) (end 6 2.77) (layer Edge.Cuts) (width 0.15))
+    (fp_line (start -7.3 0.42) (end -7.3 2.82) (layer Edge.Cuts) (width 0.15))
+    (fp_line (start -7.3 2.82) (end 6.5 2.82) (layer Edge.Cuts) (width 0.15))
+    (fp_line (start -7.3 0.42) (end 6.5 0.42) (layer Edge.Cuts) (width 0.15))
+    (fp_line (start 6.5 0.42) (end 6.5 2.82) (layer Edge.Cuts) (width 0.15))
   )
   (gr_text SONG (at 193.675 115.57) (layer F.SilkS)
