File: led-matrix.sch (KiCad schematic (older format))
At the start: 32 parts

Commit message: renumbered pcb
Parts:
- renumbered LED401 to LED1, LED414 to LED10, LED415 to LED11, LED416 to LED12, LED405 to LED13, LED406 to LED14, LED417 to LED15, LED418 to LED16, LED419 to LED17, LED420 to LED18, LED421 to LED19, LED402 to LED2, LED422 to LED20, LED423 to LED21, LED424 to LED22, LED407 to LED23, LED408 to LED24, LED425 to LED25, LED426 to LED26, LED427 to LED27, LED428 to LED28, LED429 to LED29, LED403 to LED3, LED430 to LED30, LED431 to LED31, LED432 to LED32, LED404 to LED4, LED409 to LED5, LED410 to LED6, LED411 to LED7, LED412 to LED8, LED413 to LED9
Changed lines of the file:
@@
 $EndDescr
 $Comp
-L LED_Dual_ACA LED401
+L LED_Dual_ACA LED1
 U 1 1 59DAB354
 P 2400 1900
-F 0 "LED401" H 2400 2125 50  0000 C CNN
+F 0 "LED1" H 2400 2125 50  0000 C CNN
 F 1 "LTL1BEKVJNN" H 2400 1650 50  0000 C CNN
 F 2 "w_led:LTL1BEKVJNN" H 2400 1900 50  0001 C CNN
@@
 $EndComp
 $Comp
-L LED_Dual_ACA LED409
+L LED_Dual_ACA LED5
 U 1 1 59DAB3C2
 P 2400 2700
-F 0 "LED409" H 2400 2925 50  0000 C CNN
+F 0 "LED5" H 2400 2925 50  0000 C CNN
 F 1 "LTL1BEKVJNN" H 2400 2450 50  0000 C CNN
 F 2 "w_led:LTL1BEKVJNN" H 2400 2700 50  0001 C CNN
@@
 $EndComp
 $Comp
-L LED_Dual_ACA LED417
+L LED_Dual_ACA LED15
 U 1 1 59DAB418
 P 2400 3500
-F 0 "LED417" H 2400 3725 50  0000 C CNN
+F 0 "LED15" H 2400 3725 50  0000 C CNN
 F 1 "LTL1BEKVJNN" H 2400 3250 50  0000 C CNN
 F 2 "w_led:LTL1BEKVJNN" H 2400 3500 50  0001 C CNN
@@
 $EndComp
 $Comp
-L LED_Dual_ACA LED425
+L LED_Dual_ACA LED25
 U 1 1 59DAB41E
 P 2400 4300
-F 0 "LED425" H 2400 4525 50  0000 C CNN
+F 0 "LED25" H 2400 4525 50  0000 C CNN
 F 1 "LTL1BEKVJNN" H 2400 4050 50  0000 C CNN
 F 2 "w_led:LTL1BEKVJNN" H 2400 4300 50  0001 C CNN
@@
 $EndComp
 $Comp
-L LED_Dual_ACA LED402
+L LED_Dual_ACA LED2
 U 1 1 59DAB4C6
 P 3300 1900
-F 0 "LED402" H 3300 2125 50  0000 C CNN
+F 0 "LED2" H 3300 2125 50  0000 C CNN
 F 1 "LTL1BEKVJNN" H 3300 1650 50  0000 C CNN
 F 2 "w_led:LTL1BEKVJNN" H 3300 1900 50  0001 C CNN
@@
 $EndComp
 $Comp
-L LED_Dual_ACA LED410
+L LED_Dual_ACA LED6
 U 1 1 59DAB4CC
 P 3300 2700
-F 0 "LED410" H 3300 2925 50  0000 C CNN
+F 0 "LED6" H 3300 2925 50  0000 C CNN
 F 1 "LTL1BEKVJNN" H 3300 2450 50  0000 C CNN
 F 2 "w_led:LTL1BEKVJNN" H 3300 2700 50  0001 C CNN
@@
 $EndComp
 $Comp
-L LED_Dual_ACA LED418
+L LED_Dual_ACA LED16
 U 1 1 59DAB4D2
 P 3300 3500
-F 0 "LED418" H 3300 3725 50  0000 C CNN
+F 0 "LED16" H 3300 3725 50  0000 C CNN
 F 1 "LTL1BEKVJNN" H 3300 3250 50  0000 C CNN
 F 2 "w_led:LTL1BEKVJNN" H 3300 3500 50  0001 C CNN
@@
 $EndComp
 $Comp
-L LED_Dual_ACA LED426
+L LED_Dual_ACA LED26
 U 1 1 59DAB4D8
 P 3300 4300
-F 0 "LED426" H 3300 4525 50  0000 C CNN
+F 0 "LED26" H 3300 4525 50  0000 C CNN
 F 1 "LTL1BEKVJNN" H 3300 4050 50  0000 C CNN
 F 2 "w_led:LTL1BEKVJNN" H 3300 4300 50  0001 C CNN
@@
 $EndComp
 $Comp
-L LED_Dual_ACA LED403
+L LED_Dual_ACA LED3
 U 1 1 59DAB5EE
 P 4200 1900
-F 0 "LED403" H 4200 2125 50  0000 C CNN
+F 0 "LED3" H 4200 2125 50  0000 C CNN
 F 1 "LTL1BEKVJNN" H 4200 1650 50  0000 C CNN
 F 2 "w_led:LTL1BEKVJNN" H 4200 1900 50  0001 C CNN
@@
 $EndComp
 $Comp
-L LED_Dual_ACA LED411
+L LED_Dual_ACA LED7
 U 1 1 59DAB5F4
 P 4200 2700
-F 0 "LED411" H 4200 2925 50  0000 C CNN
+F 0 "LED7" H 4200 2925 50  0000 C CNN
 F 1 "LTL1BEKVJNN" H 4200 2450 50  0000 C CNN
 F 2 "w_led:LTL1BEKVJNN" H 4200 2700 50  0001 C CNN
@@
 $EndComp
 $Comp
-L LED_Dual_ACA LED419
+L LED_Dual_ACA LED17
 U 1 1 59DAB5FA
 P 4200 3500
-F 0 "LED419" H 4200 3725 50  0000 C CNN
+F 0 "LED17" H 4200 3725 50  0000 C CNN
 F 1 "LTL1BEKVJNN" H 4200 3250 50  0000 C CNN
 F 2 "w_led:LTL1BEKVJNN" H 4200 3500 50  0001 C CNN
@@
 $EndComp
 $Comp
-L LED_Dual_ACA LED427
+L LED_Dual_ACA LED27
 U 1 1 59DAB600
 P 4200 4300
-F 0 "LED427" H 4200 4525 50  0000 C CNN
+F 0 "LED27" H 4200 4525 50  0000 C CNN
 F 1 "LTL1BEKVJNN" H 4200 4050 50  0000 C CNN
 F 2 "w_led:LTL1BEKVJNN" H 4200 4300 50  0001 C CNN
@@
 $EndComp
 $Comp
-L LED_Dual_ACA LED404
+L LED_Dual_ACA LED4
 U 1 1 59DAB606
 P 5100 1900
-F 0 "LED404" H 5100 2125 50  0000 C CNN
+F 0 "LED4" H 5100 2125 50  0000 C CNN
 F 1 "LTL1BEKVJNN" H 5100 1650 50  0000 C CNN
 F 2 "w_led:LTL1BEKVJNN" H 5100 1900 50  0001 C CNN
@@
 $EndComp
 $Comp
-L LED_Dual_ACA LED412
+L LED_Dual_ACA LED8
 U 1 1 59DAB60C
 P 5100 2700
-F 0 "LED412" H 5100 2925 50  0000 C CNN
+F 0 "LED8" H 5100 2925 50  0000 C CNN
 F 1 "LTL1BEKVJNN" H 5100 2450 50  0000 C CNN
 F 2 "w_led:LTL1BEKVJNN" H 5100 2700 50  0001 C CNN
@@
 $EndComp
 $Comp
-L LED_Dual_ACA LED420
+L LED_Dual_ACA LED18
 U 1 1 59DAB612
 P 5100 3500
-F 0 "LED420" H 5100 3725 50  0000 C CNN
+F 0 "LED18" H 5100 3725 50  0000 C CNN
 F 1 "LTL1BEKVJNN" H 5100 3250 50  0000 C CNN
 F 2 "w_led:LTL1BEKVJNN" H 5100 3500 50  0001 C CNN
@@
 $EndComp
 $Comp
-L LED_Dual_ACA LED428
+L LED_Dual_ACA LED28
 U 1 1 59DAB618
 P 5100 4300
-F 0 "LED428" H 5100 4525 50  0000 C CNN
+F 0 "LED28" H 5100 4525 50  0000 C CNN
 F 1 "LTL1BEKVJNN" H 5100 4050 50  0000 C CNN
 F 2 "w_led:LTL1BEKVJNN" H 5100 4300 50  0001 C CNN
@@
 $EndComp
 $Comp
-L LED_Dual_ACA LED405
+L LED_Dual_ACA LED13
 U 1 1 59DAB7AE
 P 6000 1900
-F 0 "LED405" H 6000 2125 50  0000 C CNN
+F 0 "LED13" H 6000 2125 50  0000 C CNN
 F 1 "LTL1BEKVJNN" H 6000 1650 50  0000 C CNN
 F 2 "w_led:LTL1BEKVJNN" H 6000 1900 50  0001 C CNN
@@
 $EndComp
 $Comp
-L LED_Dual_ACA LED413
+L LED_Dual_ACA LED9
 U 1 1 59DAB7B4
 P 6000 2700
-F 0 "LED413" H 6000 2925 50  0000 C CNN
+F 0 "LED9" H 6000 2925 50  0000 C CNN
 F 1 "LTL1BEKVJNN" H 6000 2450 50  0000 C CNN
 F 2 "w_led:LTL1BEKVJNN" H 6000 2700 50  0001 C CNN
@@
 $EndComp
 $Comp
-L LED_Dual_ACA LED421
+L LED_Dual_ACA LED19
 U 1 1 59DAB7BA
 P 6000 3500
-F 0 "LED421" H 6000 3725 50  0000 C CNN
+F 0 "LED19" H 6000 3725 50  0000 C CNN
 F 1 "LTL1BEKVJNN" H 6000 3250 50  0000 C CNN
 F 2 "w_led:LTL1BEKVJNN" H 6000 3500 50  0001 C CNN
@@
 $EndComp
 $Comp
-L LED_Dual_ACA LED429
+L LED_Dual_ACA LED29
 U 1 1 59DAB7C0
 P 6000 4300
-F 0 "LED429" H 6000 4525 50  0000 C CNN
+F 0 "LED29" H 6000 4525 50  0000 C CNN
 F 1 "LTL1BEKVJNN" H 6000 4050 50  0000 C CNN
 F 2 "w_led:LTL1BEKVJNN" H 6000 4300 50  0001 C CNN
@@
 $EndComp
 $Comp
-L LED_Dual_ACA LED406
+L LED_Dual_ACA LED14
 U 1 1 59DAB7C6
 P 6900 1900
-F 0 "LED406" H 6900 2125 50  0000 C CNN
+F 0 "LED14" H 6900 2125 50  0000 C CNN
 F 1 "LTL1BEKVJNN" H 6900 1650 50  0000 C CNN
 F 2 "w_led:LTL1BEKVJNN" H 6900 1900 50  0001 C CNN
@@
 $EndComp
 $Comp
-L LED_Dual_ACA LED414
+L LED_Dual_ACA LED10
 U 1 1 59DAB7CC
 P 6900 2700
-F 0 "LED414" H 6900 2925 50  0000 C CNN
+F 0 "LED10" H 6900 2925 50  0000 C CNN
 F 1 "LTL1BEKVJNN" H 6900 2450 50  0000 C CNN
 F 2 "w_led:LTL1BEKVJNN" H 6900 2700 50  0001 C CNN
@@
 $EndComp
 $Comp
-L LED_Dual_ACA LED422
+L LED_Dual_ACA LED20
 U 1 1 59DAB7D2
 P 6900 3500
-F 0 "LED422" H 6900 3725 50  0000 C CNN
+F 0 "LED20" H 6900 3725 50  0000 C CNN
 F 1 "LTL1BEKVJNN" H 6900 3250 50  0000 C CNN
 F 2 "w_led:LTL1BEKVJNN" H 6900 3500 50  0001 C CNN
@@
 $EndComp
 $Comp
-L LED_Dual_ACA LED430
+L LED_Dual_ACA LED30
 U 1 1 59DAB7D8
 P 6900 4300
-F 0 "LED430" H 6900 4525 50  0000 C CNN
+F 0 "LED30" H 6900 4525 50  0000 C CNN
 F 1 "LTL1BEKVJNN" H 6900 4050 50  0000 C CNN
 F 2 "w_led:LTL1BEKVJNN" H 6900 4300 50  0001 C CNN
@@
 $EndComp
 $Comp
-L LED_Dual_ACA LED407
+L LED_Dual_ACA LED23
 U 1 1 59DAB7DE
 P 7800 1900
-F 0 "LED407" H 7800 2125 50  0000 C CNN
+F 0 "LED23" H 7800 2125 50  0000 C CNN
 F 1 "LTL1BEKVJNN" H 7800 1650 50  0000 C CNN
 F 2 "w_led:LTL1BEKVJNN" H 7800 1900 50  0001 C CNN
@@
 $EndComp
 $Comp
-L LED_Dual_ACA LED415
+L LED_Dual_ACA LED11
 U 1 1 59DAB7E4
 P 7800 2700
-F 0 "LED415" H 7800 2925 50  0000 C CNN
+F 0 "LED11" H 7800 2925 50  0000 C CNN
 F 1 "LTL1BEKVJNN" H 7800 2450 50  0000 C CNN
 F 2 "w_led:LTL1BEKVJNN" H 7800 2700 50  0001 C CNN
@@
 $EndComp
 $Comp
-L LED_Dual_ACA LED423
+L LED_Dual_ACA LED21
 U 1 1 59DAB7EA
 P 7800 3500
-F 0 "LED423" H 7800 3725 50  0000 C CNN
+F 0 "LED21" H 7800 3725 50  0000 C CNN
 F 1 "LTL1BEKVJNN" H 7800 3250 50  0000 C CNN
 F 2 "w_led:LTL1BEKVJNN" H 7800 3500 50  0001 C CNN
@@
 $EndComp
 $Comp
-L LED_Dual_ACA LED431
+L LED_Dual_ACA LED31
 U 1 1 59DAB7F0
 P 7800 4300
-F 0 "LED431" H 7800 4525 50  0000 C CNN
+F 0 "LED31" H 7800 4525 50  0000 C CNN
 F 1 "LTL1BEKVJNN" H 7800 4050 50  0000 C CNN
 F 2 "w_led:LTL1BEKVJNN" H 7800 4300 50  0001 C CNN
@@
 $EndComp
 $Comp
-L LED_Dual_ACA LED408
+L LED_Dual_ACA LED24
 U 1 1 59DAB7F6
 P 8700 1900
-F 0 "LED408" H 8700 2125 50  0000 C CNN
+F 0 "LED24" H 8700 2125 50  0000 C CNN
 F 1 "LTL1BEKVJNN" H 8700 1650 50  0000 C CNN
 F 2 "w_led:LTL1BEKVJNN" H 8700 1900 50  0001 C CNN
@@
 $EndComp
 $Comp
-L LED_Dual_ACA LED416
+L LED_Dual_ACA LED12
 U 1 1 59DAB7FC
 P 8700 2700
-F 0 "LED416" H 8700 2925 50  0000 C CNN
+F 0 "LED12" H 8700 2925 50  0000 C CNN
 F 1 "LTL1BEKVJNN" H 8700 2450 50  0000 C CNN
 F 2 "w_led:LTL1BEKVJNN" H 8700 2700 50  0001 C CNN
@@
 $EndComp
 $Comp
-L LED_Dual_ACA LED424
+L LED_Dual_ACA LED22
 U 1 1 59DAB802
 P 8700 3500
-F 0 "LED424" H 8700 3725 50  0000 C CNN
+F 0 "LED22" H 8700 3725 50  0000 C CNN
 F 1 "LTL1BEKVJNN" H 8700 3250 50  0000 C CNN
 F 2 "w_led:LTL1BEKVJNN" H 8700 3500 50  0001 C CNN
@@
 $EndComp
 $Comp
-L LED_Dual_ACA LED432
+L LED_Dual_ACA LED32
 U 1 1 59DAB808
 P 8700 4300
-F 0 "LED432" H 8700 4525 50  0000 C CNN
+F 0 "LED32" H 8700 4525 50  0000 C CNN
 F 1 "LTL1BEKVJNN" H 8700 4050 50  0000 C CNN
 F 2 "w_led:LTL1BEKVJNN" H 8700 4300 50  0001 C CNN
