File: led-matrix.sch (KiCad schematic (older format))
At the start: 32 parts

Commit message: cleaned up schematics
Other:
- note added: "LED MATRIX"
Changed lines of the file:
@@
 Sheet 5 8
 Title "per|former eurorack sequencer"
-Date "2018-08-26"
-Rev "0.3"
+Date "2018-10-09"
+Rev "1.0"
 Comp "westlicht"
 Comment1 "cc-by-sa"
@@
 Connection ~ 9100 4000
 Connection ~ 9100 4600
+Wire Notes Line
+	600  600  600  6400
+Wire Notes Line
+	600  6400 11100 6400
+Wire Notes Line
+	11100 6400 11100 600
+Wire Notes Line
+	11100 600  600  600
+Text Notes 700  6300 0    51   ~ 0
+LED MATRIX
 $EndSCHEMATC

Commit message: updated schematics to kicad5
Parts:
- LED1, LED10, LED11, LED12, LED13, LED14, LED15, LED16, LED17, LED18, LED19, LED2, LED20, LED21, LED22, LED23, LED24, LED25, LED26, LED27, LED28, LED29, LED3, LED30, LED31, LED32, LED4, LED5, LED6, LED7, LED8, LED9: symbol LED_Dual_ACA -> Device:LED_Dual_ACA
