File: global.sch (KiCad schematic (older format))
At the start: 37 parts, among them Q5 MMBT3904, U11 74HC165, U12 74HC595, U13 74HC595, U14 74HC595, U5 74HCT125

Commit message: updated schematics to kicad5
Parts:
- C43, C44, C45, C49, C6: symbol C -> Device:C
- ENC1: symbol ALPS-STEC12E08 -> w_rotary_encoder:ALPS-STEC12E08
- JP1: symbol USB_A -> Connector:USB_A
- JP2: symbol Micro_SD_Card -> Connector:Micro_SD_Card
- JP3: symbol NHD-3.12-25664UC -> w_lcd:NHD-3.12-25664UC
- Q5: symbol MMBT3904 -> Transistor_BJT:MMBT3904
- R10, R11, R12, R13, R36, R49, R50, R55, R58, R61, R66, R67, R69, R70, R71, R72, R73, R74, R75, R76, R77, R9: symbol R -> Device:R
- U11: symbol 74HC165 -> w_logic:74HC165
- U12, U13, U14: symbol 74HC595 -> w_logic:74HC595
- U5: symbol 74HCT125 -> w_logic:74HCT125

Commit message: updated footprints to kicad5
Parts:
- Q5: footprint TO_SOT_Packages_SMD:SOT-23 -> Package_TO_SOT_SMD:SOT-23
- U11, U12, U13, U14: footprint Housings_SOIC:SOIC-16_3.9x9.9mm_Pitch1.27mm -> Package_SO:SOIC-16_3.9x9.9mm_P1.27mm
- U5: footprint Housings_SOIC:SOIC-14_3.9x8.7mm_Pitch1.27mm -> Package_SO:SOIC-14_3.9x8.7mm_P1.27mm
Changed lines of the file:
@@
 F 0 "U11" H 4600 4450 60  0000 C CNN
 F 1 "74HC165" H 4600 5450 60  0000 C CNN
-F 2 "Housings_SOIC:SOIC-16_3.9x9.9mm_Pitch1.27mm" H 4100 5300 60  0001 C CNN
+F 2 "Package_SO:SOIC-16_3.9x9.9mm_P1.27mm" H 4100 5300 60  0001 C CNN
 F 3 "https://octopart.com/click/track?ct=datasheets&hlid=24916538&ppid=35776&sid=370&sig=03765d0" H 4100 5300 60  0001 C CNN
 F 4 "Texas Instruments" H 4600 4550 50  0001 C CNN "MFN"
@@
 F 0 "U12" H 4600 250 60  0000 C CNN
 F 1 "74HC595" H 4600 1250 60  0000 C CNN
-F 2 "Housings_SOIC:SOIC-16_3.9x9.9mm_Pitch1.27mm" H 4100 1100 60  0001 C CNN
+F 2 "Package_SO:SOIC-16_3.9x9.9mm_P1.27mm" H 4100 1100 60  0001 C CNN
 F 3 "https://octopart.com/click/track?ct=datasheets&hlid=24917219&ppid=44183&sid=370&sig=036bbbe" H 4100 1100 60  0001 C CNN
 F 4 "Texas Instruments" H 4600 350 50  0001 C CNN "MFN"
@@
 F 0 "U13" H 4600 1650 60  0000 C CNN
 F 1 "74HC595" H 4600 2650 60  0000 C CNN
-F 2 "Housings_SOIC:SOIC-16_3.9x9.9mm_Pitch1.27mm" H 4100 2500 60  0001 C CNN
+F 2 "Package_SO:SOIC-16_3.9x9.9mm_P1.27mm" H 4100 2500 60  0001 C CNN
 F 3 "https://octopart.com/click/track?ct=datasheets&hlid=24917219&ppid=44183&sid=370&sig=036bbbe" H 4100 2500 60  0001 C CNN
 F 4 "Texas Instruments" H 4600 1750 50  0001 C CNN "MFN"
@@
 F 0 "U14" H 4600 3050 60  0000 C CNN
 F 1 "74HC595" H 4600 4050 60  0000 C CNN
-F 2 "Housings_SOIC:SOIC-16_3.9x9.9mm_Pitch1.27mm" H 4100 3900 60  0001 C CNN
+F 2 "Package_SO:SOIC-16_3.9x9.9mm_P1.27mm" H 4100 3900 60  0001 C CNN
 F 3 "https://octopart.com/click/track?ct=datasheets&hlid=24917219&ppid=44183&sid=370&sig=036bbbe" H 4100 3900 60  0001 C CNN
 F 4 "Texas Instruments" H 4600 3150 50  0001 C CNN "MFN"
@@
 F 0 "U5" H 2100 -50 60  0000 C CNN
 F 1 "74HCT125" H 2100 1150 60  0000 C CNN
-F 2 "Housings_SOIC:SOIC-14_3.9x8.7mm_Pitch1.27mm" H 2050 1100 60  0001 C CNN
+F 2 "Package_SO:SOIC-14_3.9x8.7mm_P1.27mm" H 2050 1100 60  0001 C CNN
 F 3 "https://octopart.com/click/track?ct=datasheets&hlid=24917456&ppid=464455&sid=370&sig=085083f" H 2050 1100 60  0001 C CNN
 F 4 "Texas Instruments" H 1600 1000 60  0001 C CNN "MFN"
@@
 F 0 "Q5" H 2800 2975 50  0000 L CNN
 F 1 "MMBT3904" H 2800 2900 50  0000 L CNN
-F 2 "TO_SOT_Packages_SMD:SOT-23" H 2800 2825 50  0001 L CIN
+F 2 "Package_TO_SOT_SMD:SOT-23" H 2800 2825 50  0001 L CIN
 F 3 "http://datasheet.octopart.com/MMBT3904LT1G-ON-Semiconductor-datasheet-11971584.pdf" H 2600 2900 50  0001 L CNN
 F 4 "ON Semiconductor" H 2800 3075 50  0001 C CNN "MFN"
